File: MyProject/SFT_MainBoard1.0v/SFT_MainBoard1.0v.brd (EAGLE design)
At the start: 100 x 80 mm, 42 parts, among them CN1A ZH, CN1B PH, CN1C XH, CN2A ZH, CN2B PH, CN2C XH, J1 2DC-0005X, M1 SBDBT, X1 ZH04, X2 ZH04, X3 ZH04, X9 ZH

Commit message: TETUYA KOUSIN
Parts:
- removed C4: (no value), 02_C:1608
- removed C5: (no value), 02_C:3225
- removed CN1A, CN2A: ZH, jst:B6B-ZR
- removed CN1B, CN2B: PH, jst-ph:JST-PH6
- removed CN1C, CN2C: XH, con-jst-xh:B6B-XH
- removed R11, R5, R6, R_L1, R_L2, R_L3, R_L4: (no value), 01_R:1608
- removed U$76, U$77: CHECK_0.8MM, 08_CONECTOR:CHECK_0.8MM
- removed X1, X2, X3: ZH04, con-jst:B4B-ZR
- removed X9: ZH, con-jst:B4B-ZR
- added CN1: (no value), jst-xa:B14B-XASK-1
- added CON1, CON2, CON3, CON4: I2C1, jst:B4B-ZR
- added CON5, CON6, CON7, CON8: I2C2, jst:B4B-ZR
- added R0, R1, R2, R3, R9: (no value), 01_R:1608
- added U$1, U$3, U$4: JST-PA8, jst-ph:JST-PA8
- added U$15, U$18: CHECK_0.8MM, 08_CONECTOR:CHECK_0.8MM
- moved R4 99.9 mm to (95.5, 52.0), flipped to the bottom, turned to 180 degrees
- moved J1 75.1 mm to (7.00, 12.0), turned to 0 degrees
- moved R10 55.6 mm to (18.0, 19.0), flipped to the top, turned to 0 degrees
- moved R8 31.0 mm to (69.0, 57.0), turned to 180 degrees
- moved U$78 30.1 mm to (91.0, 61.5)
- moved U$79 26.6 mm to (91.0, 59.0)
- moved LED4 19.4 mm to (96.5, 53.0)
- moved LED3 18.9 mm to (96.5, 56.0)
- moved R7 12.8 mm to (68.0, 60.0)
- moved LED2 11.4 mm to (91.5, 53.0)
- moved LED1 11.2 mm to (91.5, 56.0)
- moved C1 11.0 mm to (23.7, 5.74)
- moved U$41 6.00 mm to (44.0, 46.0)
- moved SV1 5.00 mm to (94.0, 27.8)
- moved U$2 4.00 mm to (46.0, 28.0)
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Connections:
- removed net CN1BUS3: CN1A.3, CN1B.3, CN1C.P$3, U$2.P$69
- removed net CN1BUS4: CN1A.4, CN1B.4, CN1C.P$4, U$2.P$67
- removed net CN1BUS5: CN1A.5, CN1B.5, CN1C.P$5, U$2.P$63
- removed net CN1BUS6: CN1A.6, CN1B.6, CN1C.P$6, U$2.P$61
- new net +5V: CON1.2, CON2.2, CON3.2, CON4.2, CON5.2, CON6.2, CON7.2, CON8.2, R10.2, R7.2, R8.2, R9.2
- new net N$10: CON5.3, CON6.3, CON7.3, CON8.3, R9.1, U$18.P$1
- new net N$11: CON5.4, CON6.4, CON7.4, CON8.4, R10.1, U$15.P$1
- new net N$6: CON1.1, CON2.1, CON3.1, CON4.1
- new net N$7: CON5.1, CON6.1, CON7.1, CON8.1
- new net N$8: CON1.3, CON2.3, CON3.3, CON4.3, R8.1, U$79.P$1
- new net N$9: CON1.4, CON2.4, CON3.4, CON4.4, R7.1, U$78.P$1
- net +3.3V: no longer CN1A.2, CN1B.2, CN1C.P$2, CN2A.2, CN2B.2, CN2C.P$2, R4.2, R5.2, R6.2, R7.2, X1.2, X2.2, X3.2, X9.2
- net CN2BUS3: no longer CN2A.3, CN2B.3, CN2C.P$3
- net CN2BUS4: no longer CN2A.4, CN2B.4, CN2C.P$4
- net CN2BUS5: no longer CN2A.5, CN2B.5, CN2C.P$5
- net CN2BUS6: no longer CN2A.6, CN2B.6, CN2C.P$6
- net GND: now also R0.1, R1.1, R2.1, R3.1, R4.1; no longer C4.P$2, C5.P$2, CN1A.1, CN1B.1, CN1C.P$1, CN2A.1, CN2B.1, CN2C.P$1, R8.1, R_L1.1, R_L2.1, R_L3.1, R_L4.1, X1.1, X2.1, X3.1, X9.1
- net N$1: now also R0.2; no longer R8.2
- net N$2: now also R1.2; no longer R_L1.2
- net N$3: now also R2.2; no longer R_L3.2
- net N$4: now also R3.2; no longer R_L4.2
- net N$5: now also R4.2; no longer R_L2.2
- net P12_6: no longer R5.1, U$77.P$1, X1.4, X2.4, X3.4
- net P1_6: no longer R4.1, U$76.P$1, X1.3, X2.3, X3.3
- net P3_0: no longer R10.2
- net P3_2: no longer R10.1
- net P3_5: no longer R11.2
- net P3_7: no longer R11.1
- net P6_1: no longer R6.1, U$78.P$1, X9.3
- net P6_3: no longer R7.1, U$79.P$1, X9.4
- net V_BATT: no longer C4.P$1, C5.P$1
Routing:
- net +3.3V: track 47.8 -> 0.00 mm
- net GND: track 28.2 -> 0.00 mm
Other:
- board size 100 x 80 mm -> 100 x 65 mm
- board text added: "I2C2"

Commit message: baitomae
Parts:
- removed J1: 2DC-0005X, marushin:2DC-0005D
- removed LED2, LED4: CHIPLED, 10_LED:1608
- removed R12, R3, R4: (no value), 01_R:1608
- removed U$1, U$3, U$4: JST-PA8, jst-ph:JST-PA8
- added CN2: (no value), jst-ph:B4B-PH-K-S
- added CN3, CN4, CN5: JST-PA8, jst-ph:JST-PA8
- added CN7: (no value), jst-ph:B2B-PH-K-S
- added CON9: B4B-ZR, jst:B4B-ZR
- added U$16, U$17: I2C_FXMA2102, 04_IC:DIL08
- added U$33: SS12D01G4, 09_1_switch:SS12D01G4
- added U$37, U$38, U$39: CHECK_0.8MM, 08_CONECTOR:CHECK_0.8MM
- added U$52: NJM2845, 04_IC:TO252
- moved C3 57.2 mm to (34.3, 4.73)
- moved R2 35.9 mm to (59.9, 54.6)
- moved LED3 32.2 mm to (64.5, 59.4)
- moved R1 31.5 mm to (60.0, 53.4)
- moved CON1 28.5 mm to (96.0, 51.3), turned to 90 degrees
- moved LED1 25.6 mm to (66.0, 57.8)
- moved CON2 21.8 mm to (91.0, 51.3), turned to 90 degrees
- moved R7 20.0 mm to (87.9, 62.6)
- moved U$82 18.4 mm to (2.00, 44.0)
- moved R0 18.4 mm to (43.0, 30.0)
- moved R9 18.0 mm to (5.00, 12.0)
- moved U$41 17.9 mm to (52.0, 30.0)
- moved U$15 17.1 mm to (2.00, 15.0)
- moved U$18 16.5 mm to (2.00, 12.0)
- moved R8 14.9 mm to (82.8, 62.7)
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Connections:
- net CN2BUS3 renamed P15_5
- net CN2BUS4 renamed P15_4
- removed net CN2BUS5: U$2.P$37
- removed net CN2BUS6: U$2.P$35
- removed net N$4: LED4.2, R3.2
- removed net N$6: CON1.1, CON2.1, CON3.1, CON4.1
- removed net N$7: CON5.1, CON6.1, CON7.1, CON8.1
- new net CN3: CN4.4
- new net N$13: CN5.4
- new net NC1: SV1.4
- new net NC2: CN3.4
- new net P5_1: U$2.P$63
- new net P5_3: U$2.P$61
- new net P6_0: U$16.2, U$2.P$35
- new net P6_2: U$16.4, U$2.P$37
- new net P6_5: M1.7, U$2.P$69, U$82.P$1
- new net P6_7: M1.9, U$2.P$67
- new net V2: CON1.2, CON2.2, CON3.2, CON4.2, R7.2, R8.2, U$16.8, U$33.2
- net +3.3V: now also CN3.3, CN4.3, CN5.3, SV1.3, U$16.1, U$17.1, U$33.1, U$52.3; no longer R12.2
- net +5V: now also CN3.2, CN4.2, CN5.2, CN7.2, SV1.2, U$17.8, U$33.3, U$52.1; no longer CON1.2, CON2.2, CON3.2, CON4.2, R7.2, R8.2
- net GND: now also CN1.1, CN3.1, CN4.1, CN5.1, CN7.1, CON1.1, CON2.1, CON3.1, CON4.1, CON5.1, CON6.1, CON7.1, CON8.1, SV1.1, U$16.5, U$17.5, U$37.P$1, U$38.P$1, U$39.P$1, U$52.2; no longer J1.2, R3.1, R4.1
- net N$10: now also U$17.7
- net N$11: now also U$17.6
- net N$5: now also CN1.2; no longer LED2.2, R4.2
- net N$8: now also U$16.7
- net N$9: now also U$16.6
- net P0_0: now also CN1.11, SV1.13
- net P0_1: now also CN1.12, SV1.14
- net P0_2: now also CN1.13, SV1.15
- net P0_3: now also CN1.14, SV1.16
- net P0_4: now also SV1.17
- net P0_5: now also SV1.18
- net P0_6: now also SV1.19
- net P0_7: now also SV1.20
- net P12_0: now also SV1.21
- net P12_1: now also SV1.22; no longer J1.3, R12.1
- net P12_2: now also SV1.23
- net P12_3: now also SV1.24; no longer U$41.P$2
- net P1_4: now also CN5.5
- net P1_5: now also CN5.6
- net P1_6: now also CN5.7
- net P1_7: now also CN5.8
- net P2_0: now also CN3.5
- net P2_1: now also CN3.6; no longer M1.6
- net P2_2: now also CN3.7
- net P2_3: now also CN3.8; no longer M1.7, U$82.P$1
- net P2_4: now also CN4.5
- net P2_5: now also CN4.6; no longer M1.8, U$83.P$1
- net P2_6: now also CN4.7
- net P2_7: now also CN4.8; no longer M1.9
- net P3_0: now also CN1.3, SV1.5
- net P3_1: now also CN1.4, SV1.6
- net P3_2: now also CN1.5, SV1.7
- net P3_3: now also CN1.6, SV1.8
- net P3_4: now also CN1.7, SV1.9
- net P3_5: now also CN1.8, SV1.10
- net P3_6: now also CN1.9, SV1.11
- net P3_7: now also CN1.10, SV1.12
- net P4_0: now also U$41.P$2
- net P4_2: now also SV1.25
- net P4_3: now also SV1.26
- net P4_4: no longer LED4.1
- net P4_6: no longer LED2.1
- net P5_4: now also U$17.2
- net P5_5: now also U$17.3
- net P5_6: now also U$17.4
- net P6_1: now also U$16.3
- net P6_4: now also M1.6
- net P6_6: now also M1.8, U$83.P$1
- net V_DDIN: no longer J1.1
Routing:
- net P0_5: track 0.00 -> 60.2 mm, vias 0 -> 1
- net P6_5: track 0.00 -> 55.8 mm
- net P1_6: track 0.00 -> 55.7 mm
- net P1_7: track 0.00 -> 53.6 mm
- net P1_4: track 0.00 -> 51.2 mm
- net P0_4: track 0.00 -> 50.8 mm
- net P1_5: track 0.00 -> 49.4 mm
- net V2: track 0.00 -> 48.0 mm
- net P6_6: track 0.00 -> 41.9 mm
- net P0_3: track 0.00 -> 40.9 mm
- net P12_0: track 0.00 -> 40.0 mm
- net P0_2: track 0.00 -> 39.9 mm, vias 0 -> 1
- net P12_2: track 0.00 -> 39.3 mm
- net P12_3: track 0.00 -> 39.3 mm
- net P12_1: track 0.00 -> 39.3 mm
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Other:
- board text added: "GND"

Commit message: kannsei kana
Parts:
- removed LED1, LED3: CHIPLED, 10_LED:1608
- added BLUE, RED: CHIPLED, 10_LED:1608
- CN3, CN4, CN5: value JST-PA8 -> (none); device jst-ph:JST-PA8 -> jst-ph:B8B-PH-K-S
- moved R2 65.8 mm to (14.9, 6.65), turned to 270 degrees
- moved R1 55.7 mm to (34.0, 4.05), turned to 0 degrees
- moved C3 24.4 mm to (58.7, 3.27), turned to 0 degrees
- moved C1 9.62 mm to (15.8, 11.1), turned to 90 degrees
- moved CN5 2.00 mm to (55.0, 60.0), turned to 0 degrees
- moved CN4 1.00 mm to (35.0, 60.0), turned to 0 degrees
- moved R10 1.00 mm to (5.00, 14.0)
- moved R9 1.00 mm to (5.00, 11.0)
- moved U$15 1.00 mm to (2.00, 14.0)
- moved U$18 1.00 mm to (2.00, 11.0)
- moved U$38 1.00 mm to (3.00, 38.0)
- moved U$82 1.00 mm to (3.00, 44.0)
- moved U$83 1.00 mm to (3.00, 48.0)
- moved CN7 0.71 mm to (10.4, 3.55)
- moved CN2 0.50 mm to (77.0, 3.50)
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Connections:
- net CN3 renamed NC3
- net N$13 renamed NC4
- net +3.3V: now also CN2.2, CON9.2
- net GND: now also CN2.1, CON9.1
- net N$2: now also RED.2; no longer LED1.2
- net N$3: now also BLUE.2; no longer LED3.2
- net P12_4: now also M1.10
- net P12_5: now also CN2.3, CON9.3; no longer M1.10
- net P12_6: now also CN2.4, CON9.4, RED.1
- net P12_7: now also BLUE.1
- net P4_5: no longer LED3.1
- net P4_7: no longer LED1.1
Routing:
- net +5V: track 16.5 -> 289.1 mm, vias 0 -> 1
- net P12_6: track 0.00 -> 88.2 mm
- net P12_5: track 30.7 -> 83.0 mm, vias 0 -> 1
- net P12_4: track 0.00 -> 27.0 mm
- net P12_7: track 0.00 -> 25.6 mm, vias 0 -> 1
- net +3.3V: track 0.00 -> 17.7 mm
- net N$2: track 0.00 -> 12.3 mm, vias 0 -> 1
- net N$10: track 32.6 -> 44.8 mm
- net GND: track 4.61 -> 16.5 mm
- net N$11: track 22.7 -> 34.2 mm
- net N$3: track 0.00 -> 7.49 mm, vias 0 -> 1
- net V_DDIN: track 0.00 -> 3.34 mm
- net P1_6: track 55.7 -> 58.9 mm
- net P1_4: track 51.2 -> 54.1 mm
- net P2_3: track 18.6 -> 16.9 mm
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Other:
- board text added: "SFT MainBoard 1.0v"
- board text removed: "Troostite 1.0v"

Commit message: syukujitu syuuryou
Connections:
- net P12_6: no longer RED.1
- net P5_7: now also RED.1
Routing:
- net P12_6: track 88.2 -> 65.9 mm
- net P5_7: track 0.00 -> 14.5 mm
Changed lines of the file:
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@@
 <signal name="P12_6">
 <contactref element="U$2" pad="P$52"/>
-<contactref element="RED" pad="1"/>
 <wire x1="26.94" y1="16.542" x2="28.242" y2="15.24" width="0.3" layer="1"/>
-<wire x1="28.242" y1="15.24" x2="30.988" y2="15.24" width="0.3" layer="1"/>
-<wire x1="30.988" y1="15.24" x2="30.988" y2="5.842" width="0.3" layer="1"/>
-<wire x1="30.988" y1="5.842" x2="30.226" y2="5.08" width="0.3" layer="1"/>
-<wire x1="30.226" y1="5.08" x2="21.844" y2="5.08" width="0.3" layer="1"/>
-<wire x1="21.844" y1="5.08" x2="20.24" y2="3.476" width="0.3" layer="1"/>
-<wire x1="20.24" y1="3.476" x2="20.24" y2="2.31" width="0.3" layer="1"/>
 <contactref element="CN2" pad="4"/>
 <contactref element="CON9" pad="4"/>
@@
 <wire x1="72.42" y1="5.08" x2="60.96" y2="5.08" width="0.3" layer="1"/>
 <wire x1="60.96" y1="5.08" x2="50.8" y2="15.24" width="0.3" layer="1"/>
-<wire x1="50.8" y1="15.24" x2="30.988" y2="15.24" width="0.3" layer="1"/>
+<wire x1="50.8" y1="15.24" x2="28.242" y2="15.24" width="0.3" layer="1"/>
 <wire x1="74" y1="3.5" x2="76.23" y2="1.27" width="0.3" layer="1"/>
 <wire x1="76.23" y1="1.27" x2="83.07" y2="1.27" width="0.3" layer="1"/>
@@
 <signal name="P5_7">
 <contactref element="U$2" pad="P$47"/>
+<contactref element="RED" pad="1"/>
+<wire x1="20.24" y1="2.31" x2="20.32" y2="2.39" width="0.3" layer="1"/>
+<wire x1="20.32" y1="2.39" x2="20.32" y2="4.826" width="0.3" layer="1"/>
+<wire x1="20.32" y1="4.826" x2="25.654" y2="10.16" width="0.3" layer="1"/>
+<wire x1="25.654" y1="10.16" x2="28.178" y2="10.16" width="0.3" layer="1"/>
+<wire x1="28.178" y1="10.16" x2="29.48" y2="11.462" width="0.3" layer="1"/>
 </signal>
 <signal name="V_SSA2">

Commit message: baitomae
Connections:
- net P12_4: now also CN2.4, CON9.4; no longer M1.10
- net P12_6: now also M1.10; no longer CN2.4, CON9.4
Routing:
- net P12_4: track 27.0 -> 95.0 mm, vias 0 -> 1
- net P12_6: track 65.9 -> 46.2 mm
- net P12_5: track 83.0 -> 83.9 mm
Changed lines of the file:
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@@
 <setting verticaltext="up"/>
 </settings>
-<grid distance="0.01" unitdist="inch" unit="inch" style="lines" multiple="1" display="yes" altdistance="0.025" altunitdist="inch" altunit="inch"/>
+<grid distance="1" unitdist="mm" unit="mm" style="lines" multiple="1" display="yes" altdistance="0.025" altunitdist="inch" altunit="inch"/>
 <layers>
 <layer number="1" name="Top" color="4" fill="1" visible="yes" active="yes"/>
@@
 <signal name="P12_4">
 <contactref element="U$2" pad="P$72"/>
-<contactref element="M1" pad="10"/>
 <wire x1="26.94" y1="41.942" x2="16.338" y2="41.942" width="0.3" layer="16"/>
-<wire x1="16.338" y1="41.942" x2="4.72" y2="53.56" width="0.3" layer="16"/>
+<contactref element="CON9" pad="4"/>
+<contactref element="CN2" pad="4"/>
+<wire x1="74" y1="3.5" x2="69.88" y2="7.62" width="0.3" layer="1"/>
+<wire x1="69.88" y1="7.62" x2="60.96" y2="7.62" width="0.3" layer="1"/>
+<wire x1="60.96" y1="7.62" x2="48.768" y2="19.812" width="0.3" layer="1"/>
+<wire x1="48.768" y1="19.812" x2="48.768" y2="34.544" width="0.3" layer="1"/>
+<wire x1="48.768" y1="34.544" x2="46.736" y2="36.576" width="0.3" layer="1"/>
+<via x="46.736" y="36.576" extent="1-16" drill="0.5"/>
+<wire x1="46.736" y1="36.576" x2="34.798" y2="36.576" width="0.3" layer="16"/>
+<wire x1="34.798" y1="36.576" x2="30.734" y2="40.64" width="0.3" layer="16"/>
+<wire x1="30.734" y1="40.64" x2="28.242" y2="40.64" width="0.3" layer="16"/>
+<wire x1="28.242" y1="40.64" x2="26.94" y2="41.942" width="0.3" layer="16"/>
+<wire x1="74" y1="3.5" x2="75.5" y2="2" width="0.3" layer="1"/>
+<wire x1="75.5" y1="2" x2="83.8" y2="2" width="0.3" layer="1"/>
+<wire x1="83.8" y1="2" x2="85.5" y2="3.7" width="0.3" layer="1"/>
 </signal>
 <signal name="P12_5">
@@
 <contactref element="CON9" pad="3"/>
 <contactref element="CN2" pad="3"/>
-<wire x1="71.882" y1="10.16" x2="60.706" y2="10.16" width="0.3" layer="1"/>
-<wire x1="60.706" y1="10.16" x2="48.514" y2="22.352" width="0.3" layer="1"/>
-<wire x1="48.514" y1="22.352" x2="48.514" y2="33.02" width="0.3" layer="1"/>
-<wire x1="48.514" y1="33.02" x2="45.72" y2="35.814" width="0.3" layer="1"/>
-<via x="45.72" y="35.814" extent="1-16" drill="0.4"/>
-<wire x1="45.72" y1="35.814" x2="39.592" y2="41.942" width="0.3" layer="16"/>
-<wire x1="39.592" y1="41.942" x2="29.48" y2="41.942" width="0.3" layer="16"/>
-<wire x1="76" y1="3.5" x2="76" y2="6.042" width="0.3" layer="1"/>
-<wire x1="76" y1="6.042" x2="71.882" y2="10.16" width="0.3" layer="1"/>
 <wire x1="76" y1="3.5" x2="78.342" y2="5.842" width="0.3" layer="16"/>
 <wire x1="78.342" y1="5.842" x2="84.858" y2="5.842" width="0.3" layer="16"/>
 <wire x1="84.858" y1="5.842" x2="87" y2="3.7" width="0.3" layer="16"/>
+<wire x1="76" y1="3.5" x2="69.34" y2="10.16" width="0.3" layer="1"/>
+<wire x1="69.34" y1="10.16" x2="61.468" y2="10.16" width="0.3" layer="1"/>
+<wire x1="61.468" y1="10.16" x2="50.292" y2="21.336" width="0.3" layer="1"/>
+<wire x1="50.292" y1="21.336" x2="50.292" y2="36.068" width="0.3" layer="1"/>
+<wire x1="50.292" y1="36.068" x2="48.006" y2="38.354" width="0.3" layer="1"/>
+<via x="48.006" y="38.354" extent="1-16" drill="0.5"/>
+<wire x1="48.006" y1="38.354" x2="35.814" y2="38.354" width="0.3" layer="16"/>
+<wire x1="35.814" y1="38.354" x2="32.258" y2="41.91" width="0.3" layer="16"/>
+<wire x1="32.258" y1="41.91" x2="29.512" y2="41.91" width="0.3" layer="16"/>
+<wire x1="29.512" y1="41.91" x2="29.48" y2="41.942" width="0.3" layer="16"/>
 </signal>
 <signal name="P6_4">
@@
 <signal name="P12_6">
 <contactref element="U$2" pad="P$52"/>
-<wire x1="26.94" y1="16.542" x2="28.242" y2="15.24" width="0.3" layer="1"/>
-<contactref element="CN2" pad="4"/>
-<contactref element="CON9" pad="4"/>
-<wire x1="74" y1="3.5" x2="72.42" y2="5.08" width="0.3" layer="1"/>
-<wire x1="72.42" y1="5.08" x2="60.96" y2="5.08" width="0.3" layer="1"/>
-<wire x1="60.96" y1="5.08" x2="50.8" y2="15.24" width="0.3" layer="1"/>
-<wire x1="50.8" y1="15.24" x2="28.242" y2="15.24" width="0.3" layer="1"/>
-<wire x1="74" y1="3.5" x2="76.23" y2="1.27" width="0.3" layer="1"/>
-<wire x1="76.23" y1="1.27" x2="83.07" y2="1.27" width="0.3" layer="1"/>
-<wire x1="83.07" y1="1.27" x2="85.5" y2="3.7" width="0.3" layer="1"/>
+<contactref element="M1" pad="10"/>
+<wire x1="26.94" y1="16.542" x2="24" y2="19.482" width="0.3" layer="1"/>
+<wire x1="24" y1="19.482" x2="24" y2="31" width="0.3" layer="1"/>
+<wire x1="24" y1="31" x2="4.72" y2="50.28" width="0.3" layer="1"/>
+<wire x1="4.72" y1="50.28" x2="4.72" y2="53.56" width="0.3" layer="1"/>
 </signal>
 <signal name="P12_7">

Commit message: kyuukei reset
Parts:
- added C4, C5: (no value), 02_C:1608
- moved U$38 1.00 mm to (4.00, 38.0)
- moved U$82 1.00 mm to (4.00, 44.0)
- moved U$83 1.00 mm to (4.00, 48.0)
- renumbered U$16 to IC2, U$17 to IC1, U$41 to SP
Connections:
- removed net V_DDIN: C3.P$1, U$2.P$2
- removed net V_DDIN2: U$2.P$41
- net +3.3V: now also C5.P$1
- net +5V: now also C3.P$1, C4.P$1, U$2.P$2, U$2.P$41
- net GND: now also C4.P$2, C5.P$2
- net P12_4: now also CN2.3, CON9.3; no longer CN2.4, CON9.4
- net P12_5: now also CN2.4, CON9.4; no longer CN2.3, CON9.3
Routing:
- net +5V: track 289.1 -> 309.7 mm, vias 1 -> 2
- net +3.3V: track 17.7 -> 23.2 mm
- net V_DDIN: track 3.34 -> 0.00 mm
- net P12_5: track 83.9 -> 80.9 mm
- net P12_4: track 95.0 -> 95.9 mm
- net P6_5: track 55.1 -> 54.5 mm
Other:
- board text added: "HILLTOP"
- board text removed: "dsky"

Commit message: tetuya
Parts:
- added DRILEGEND: (no value), drilegend:DRILEGEND
Other:
- board text added: "穴図"

Commit message: test2
Parts:
- removed C4, C5: (no value), 02_C:1608
- removed DRILEGEND: (no value), drilegend:DRILEGEND
- moved U$38 1.00 mm to (3.00, 38.0)
- moved U$82 1.00 mm to (3.00, 44.0)
- moved U$83 1.00 mm to (3.00, 48.0)
- renumbered IC1 to U$17, IC2 to U$16, SP to U$41
Connections:
- new net V_DDIN: C3.P$1, U$2.P$2
- new net V_DDIN2: U$2.P$41
- net +3.3V: no longer C5.P$1
- net +5V: no longer C3.P$1, C4.P$1, U$2.P$2, U$2.P$41
- net GND: no longer C4.P$2, C5.P$2
- net P12_4: now also CN2.4, CON9.4; no longer CN2.3, CON9.3
- net P12_5: now also CN2.3, CON9.3; no longer CN2.4, CON9.4
Routing:
- net +5V: track 309.7 -> 289.1 mm, vias 2 -> 1
- net +3.3V: track 23.2 -> 17.7 mm
- net V_DDIN: track 0.00 -> 3.34 mm
- net P12_5: track 80.9 -> 83.9 mm
- net P12_4: track 95.9 -> 95.0 mm
- net P6_5: track 54.5 -> 55.1 mm
Other:
- board text added: "dsky"
- board text removed: "HILLTOP"
- board text removed: "穴図"
