File: MyProject/SFT_MainBoard1.0v/SFT_MainBoard1.0v.sch (EAGLE design)
At the start: 40 parts, among them CON1 I2C1, CON2 I2C1, CON3 I2C1, CON4 I2C1, CON5 I2C2, CON6 I2C2, CON7 I2C2, CON8 I2C2, J1 2DC-0005X, M1 SBDBT

Commit message: baitomae
Parts:
- removed J1: 2DC-0005X, marushin:2DC-0005X
- removed LED2, LED4: CHIPLED, 10_LED:CHIPLED
- removed R12, R3, R4: (no value), 01_R:RESISTOR__SMD
- removed U$3: JST-PA8, jst-ph:JST-PA8
- added CN2: (no value), jst-ph:B4B-PH-K-S
- added CN5: JST-PA8, jst-ph:JST-PA8
- added CN7: (no value), jst-ph:B2B-PH-K-S
- added CON9: B4B-ZR, jst:B4B-ZR
- added U$16, U$17: I2C_FXMA2102, 04_IC:I2C_FXMA2102
- added U$33: SS12D01G4, 09_1_switch:SS12D01G4
- added U$37, U$38, U$39: CHECK_0.8MM, 08_CONECTOR:CHECK_0.8MM
- added U$52: NJM2845, 04_IC:NJM2845
- renumbered U$1 to CN3, U$4 to CN4
Connections:
- net CN2BUS3 renamed P15_5
- net CN2BUS4 renamed P15_4
- removed net CN2BUS5: U$2.P$37
- removed net CN2BUS6: U$2.P$35
- removed net N$4: LED4.K, R3.P$2
- removed net N$6: CON1.1, CON2.1, CON3.1, CON4.1
- removed net N$7: CON5.1, CON6.1, CON7.1, CON8.1
- new net CN3: CN4.4
- new net N$13: CN5.4
- new net NC1: SV1.4
- new net NC2: CN3.4
- new net P5_1: U$2.P$63
- new net P5_3: U$2.P$61
- new net P6_0: U$16.A0, U$2.P$35
- new net P6_2: U$16.OE, U$2.P$37
- new net P6_5: M1.TX, U$2.P$69, U$82.P$1
- new net P6_7: M1.CTS, U$2.P$67
- new net V2: CON1.2, CON2.2, CON3.2, CON4.2, R7.P$2, R8.P$2, U$16.VCCB, U$33.P$2
- net +3.3V: now also CN3.3, CN4.3, CN5.3, SV1.3, U$16.VCCA, U$17.VCCA, U$33.P$1, U$52.VOUT; no longer R12.P$2
- net +5V: now also CN3.2, CN4.2, CN5.2, CN7.2, SV1.2, U$17.VCCB, U$33.P$3, U$52.VIN; no longer CON1.2, CON2.2, CON3.2, CON4.2, R7.P$2, R8.P$2
- net GND: now also CN1.1, CN3.1, CN4.1, CN5.1, CN7.1, CON1.1, CON2.1, CON3.1, CON4.1, CON5.1, CON6.1, CON7.1, CON8.1, SV1.1, U$16.GND, U$17.GND, U$37.P$1, U$38.P$1, U$39.P$1, U$52.G; no longer J1.S, R3.P$1, R4.P$1
- net N$10: now also U$17.B0
- net N$11: now also U$17.B1
- net N$5: now also CN1.2; no longer LED2.K, R4.P$2
- net N$8: now also U$16.B0
- net N$9: now also U$16.B1
- net P0_0: now also CN1.11, SV1.13
- net P0_1: now also CN1.12, SV1.14
- net P0_2: now also CN1.13, SV1.15
- net P0_3: now also CN1.14, SV1.16
- net P0_4: now also SV1.17
- net P0_5: now also SV1.18
- net P0_6: now also SV1.19
- net P0_7: now also SV1.20
- net P12_0: now also SV1.21
- net P12_1: now also SV1.22; no longer J1.R, R12.P$1
- net P12_2: now also SV1.23
- net P12_3: now also SV1.24; no longer U$41.PLUS
- net P1_4: now also CN5.5
- net P1_5: now also CN5.6
- net P1_6: now also CN5.7
- net P1_7: now also CN5.8
- net P2_0: now also CN3.5
- net P2_1: now also CN3.6; no longer M1.RTS
- net P2_2: now also CN3.7
- net P2_3: now also CN3.8; no longer M1.TX, U$82.P$1
- net P2_4: now also CN4.5
- net P2_5: now also CN4.6; no longer M1.RX, U$83.P$1
- net P2_6: now also CN4.7
- net P2_7: now also CN4.8; no longer M1.CTS
- net P3_0: now also CN1.3, SV1.5
- net P3_1: now also CN1.4, SV1.6
- net P3_2: now also CN1.5, SV1.7
- net P3_3: now also CN1.6, SV1.8
- net P3_4: now also CN1.7, SV1.9
- net P3_5: now also CN1.8, SV1.10
- net P3_6: now also CN1.9, SV1.11
- net P3_7: now also CN1.10, SV1.12
- net P4_0: now also U$41.PLUS
- net P4_2: now also SV1.25
- net P4_3: now also SV1.26
- net P4_4: no longer LED4.A
- net P4_6: no longer LED2.A
- net P5_4: now also U$17.A0
- net P5_5: now also U$17.A1
- net P5_6: now also U$17.OE
- net P6_1: now also U$16.A1
- net P6_4: now also M1.RTS
- net P6_6: now also M1.RX, U$83.P$1
- net V_DDIN: no longer J1.P
Other:
- moved on the sheet: CN1, CON1, CON2, CON3, CON4, R7, R8, SV1

Commit message: kannsei kana
Parts:
- removed LED3: CHIPLED, 10_LED:CHIPLED
- added BLUE: CHIPLED, 10_LED:CHIPLED
- CN3, CN4, CN5: value JST-PA8 -> (none); device jst-ph:JST-PA8 -> jst-ph:B8B-PH-K-S
- renumbered LED1 to RED
Connections:
- net CN3 renamed NC3
- net N$13 renamed NC4
- net +3.3V: now also CN2.2, CON9.2
- net GND: now also CN2.1, CON9.1
- net N$3: now also BLUE.K; no longer LED3.K
- net P12_4: now also M1.STO
- net P12_5: now also CN2.3, CON9.3; no longer M1.STO
- net P12_6: now also CN2.4, CON9.4, RED.A
- net P12_7: now also BLUE.A
- net P4_5: no longer LED3.A
- net P4_7: no longer RED.A
Other:
- note added: "for other"
- moved on the sheet: C1, C2, C3, CN2, CN7, CON9, R0, R2, U$52

Commit message: syukujitu syuuryou
Connections:
- net P12_6: no longer RED.A
- net P5_7: now also RED.A
Changed lines of the file:
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@@
-</segment>
-<segment>
-<label x="452.12" y="238.76" size="1.016" layer="95" rot="R180" xref="yes"/>
-<pinref part="RED" gate="G$1" pin="A"/>
-<wire x1="457.2" y1="238.76" x2="452.12" y2="238.76" width="0.1524" layer="91"/>
 </segment>
 <segment>
@@
 <junction x="309.88" y="233.68"/>
 </segment>
+<segment>
+<label x="452.12" y="238.76" size="1.016" layer="95" rot="R180" xref="yes"/>
+<pinref part="RED" gate="G$1" pin="A"/>
+<wire x1="457.2" y1="238.76" x2="452.12" y2="238.76" width="0.1524" layer="91"/>
+</segment>
 </net>

Commit message: baitomae
Connections:
- net P12_4: now also CN2.4, CON9.4; no longer M1.STO
- net P12_6: now also M1.STO; no longer CN2.4, CON9.4
Changed lines of the file:
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@@
 </segment>
 <segment>
-<pinref part="M1" gate="G$1" pin="STO"/>
-<wire x1="38.1" y1="368.3" x2="35.56" y2="368.3" width="0.1524" layer="91"/>
-<label x="35.56" y="368.3" size="1.016" layer="95" rot="R180" xref="yes"/>
+<pinref part="CN2" gate="G$1" pin="4"/>
+<pinref part="CON9" gate="G$1" pin="4"/>
+<wire x1="238.76" y1="309.88" x2="236.22" y2="309.88" width="0.1524" layer="91"/>
+<wire x1="259.08" y1="309.88" x2="238.76" y2="309.88" width="0.1524" layer="91"/>
+<label x="236.22" y="309.88" size="1.27" layer="95" rot="R180" xref="yes"/>
 </segment>
 </net>
@@
 </segment>
 <segment>
-<pinref part="CN2" gate="G$1" pin="4"/>
-<pinref part="CON9" gate="G$1" pin="4"/>
-<wire x1="238.76" y1="309.88" x2="236.22" y2="309.88" width="0.1524" layer="91"/>
-<wire x1="259.08" y1="309.88" x2="238.76" y2="309.88" width="0.1524" layer="91"/>
-<label x="236.22" y="309.88" size="1.27" layer="95" rot="R180" xref="yes"/>
+<pinref part="M1" gate="G$1" pin="STO"/>
+<wire x1="38.1" y1="368.3" x2="35.56" y2="368.3" width="0.1524" layer="91"/>
+<label x="35.56" y="368.3" size="1.016" layer="95" rot="R180" xref="yes"/>
 </segment>
 </net>

Commit message: kyuukei reset
Parts:
- added C4, C5: (no value), 02_C:1608
- renumbered U$16 to IC2, U$17 to IC1, U$41 to SP
Connections:
- removed net V_DDIN: C3.1, U$2.P$2
- removed net V_DDIN2: U$2.P$41
- net +3.3V: now also C5.1
- net +5V: now also C3.1, C4.1, U$2.P$2, U$2.P$41
- net GND: now also C4.2, C5.2
- net P12_4: now also CN2.3, CON9.3; no longer CN2.4, CON9.4
- net P12_5: now also CN2.4, CON9.4; no longer CN2.3, CON9.3
Other:
- note added: "I2C1"
- note added: "I2C2"
- note added: "I2C3"
- moved on the sheet: CN2, CON9

Commit message: test2
Parts:
- removed C4, C5: (no value), 02_C:1608
- renumbered IC1 to U$17, IC2 to U$16, SP to U$41
Connections:
- new net V_DDIN: C3.1, U$2.P$2
- new net V_DDIN2: U$2.P$41
- net +3.3V: no longer C5.1
- net +5V: no longer C3.1, C4.1, U$2.P$2, U$2.P$41
- net GND: no longer C4.2, C5.2
- net P12_4: now also CN2.4, CON9.4; no longer CN2.3, CON9.3
- net P12_5: now also CN2.3, CON9.3; no longer CN2.4, CON9.4
Other:
- note removed: "I2C1"
- note removed: "I2C2"
- note removed: "I2C3"
- moved on the sheet: CN2, CON9
