File: MyProject/SFT_MoterBridge_1.0v/SFT_MotorBridge.brd (EAGLE design)
At the start: 100 x 80 mm, 18 parts

Commit message: 月曜バイト行く前の更新
Parts:
- added SV1: (no value), con-ml:ML26
- added U$10, U$11, U$14, U$26, U$9: (no value), 01_R:1608
- moved OK1 90.0 mm to (67.8, 22.5), flipped to the bottom, turned to 180 degrees
- moved CN5 2.24 mm to (92.0, 31.0), turned to 90 degrees
Connections:
- removed net N$10: CN5.10
- removed net N$11: CN5.11
- removed net N$12: CN5.12
- removed net N$9: CN5.9
- new net +5V: U$10.2, U$11.2, U$14.2, U$26.2, U$9.2
- new net N$5: OK1.1, U$9.1
- new net N$6: OK1.3, U$10.1
- new net N$7: OK1.5, U$11.1
- new net N$8: OK1.7, U$14.1
- new net SPEED_OUT_1: CN5.9, OK1.16
- new net SPEED_OUT_2: CN5.10, OK1.14
- new net SPEED_OUT_3: CN5.11, OK1.12
- new net SPEED_OUT_4: CN5.12, OK1.10
- net CW_CCW_IN_1: now also SV1.5
- net CW_CCW_IN_2: now also SV1.6
- net CW_CCW_IN_3: now also SV1.7
- net CW_CCW_IN_4: now also SV1.8
- net GND: now also OK1.11, OK1.13, OK1.15, OK1.9
- net SPEED_1: now also OK1.2
- net SPEED_2: now also OK1.4
- net SPEED_3: now also OK1.6
- net SPEED_4: now also OK1.8
- net VLM_1: now also SV1.1
- net VLM_2: now also SV1.2
- net VLM_3: now also SV1.3
- net VLM_4: now also SV1.4
- net VRH_1: now also U$26.1
Routing:
- net SPEED_1: track 0.00 -> 124.0 mm
- net VRH_1: track 0.00 -> 123.4 mm, vias 0 -> 1
- net VLM_2: track 0.00 -> 120.6 mm, vias 0 -> 1
- net VLM_3: track 0.00 -> 116.7 mm, vias 0 -> 1
- net SPEED_2: track 0.00 -> 104.4 mm
- net VLM_1: track 0.00 -> 103.2 mm, vias 0 -> 1
- net VLM_4: track 0.00 -> 77.8 mm
- net CW_CCW_IN_4: track 0.00 -> 70.7 mm
- net SPEED_4: track 0.00 -> 60.0 mm, vias 0 -> 1
- net SPEED_3: track 0.00 -> 56.5 mm, vias 0 -> 2
- net CW_CCW_IN_3: track 0.00 -> 51.8 mm
- net CW_CCW_IN_2: track 0.00 -> 41.2 mm
- net CW_CCW_IN_1: track 0.00 -> 31.3 mm
- net SPEED_OUT_1: track 0.00 -> 27.9 mm
- net SPEED_OUT_2: track 0.00 -> 27.9 mm
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- added copper zone on layer 16, net GND

Commit message: 月曜バイト終了
Parts:
- removed U$10, U$11, U$14, U$26, U$9: (no value), 01_R:1608
- added F5, F6, F7, F8: CHIP_FET, 06_FET:SOT23
- added LED1, LED2, LED3, LED4: (no value), led:LED5MM
- added R0, R10, R11, R12, R13, R14, R15, R16, R17, R18, R19, R20, R9: (no value), 01_R:1608
- moved CN1 53.1 mm to (28.0, 10.0)
- moved F1 52.2 mm to (36.0, 5.00), turned to 270 degrees
- moved R1 51.5 mm to (42.0, 2.00)
- moved R2 48.5 mm to (39.0, 5.00), turned to 90 degrees
- moved R8 42.6 mm to (39.0, 50.0), turned to 90 degrees
- moved R7 39.5 mm to (42.0, 47.0)
- moved SV1 38.6 mm to (91.0, 32.0), turned to 90 degrees
- moved F4 38.2 mm to (36.0, 50.0), turned to 270 degrees
- moved CN4 37.1 mm to (28.0, 55.0)
- moved CN2 23.2 mm to (28.0, 25.0)
- moved F2 22.4 mm to (36.0, 20.0), turned to 270 degrees
- moved R3 21.8 mm to (42.0, 17.0)
- moved R4 19.3 mm to (39.0, 20.0), turned to 90 degrees
- moved OK1 18.4 mm to (62.0, 40.0)
- moved CN5 17.0 mm to (75.0, 32.0)
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Connections:
- new net N$10: F6.1, R11.2, R12.1
- new net N$11: F7.1, R13.2, R14.1
- new net N$12: F8.1, R15.2, R16.1
- new net N$9: F5.1, R10.1, R9.2
- new net RUN_BRAKE_IN_1: R10.2, SV1.13
- new net RUN_BRAKE_IN_2: R12.2, SV1.14
- new net RUN_BRAKE_IN_3: R14.2, SV1.15
- new net RUN_BRAKE_IN_4: R16.2, SV1.16
- net +5V: now also R0.2, R17.2, R18.2, R19.2, R20.2; no longer U$10.2, U$11.2, U$14.2, U$26.2, U$9.2
- net ALARM_1: now also LED1.K
- net ALARM_2: now also LED2.K
- net ALARM_3: now also LED3.K
- net ALARM_4: now also LED4.K
- net GND: now also F5.2, F6.2, F7.2, F8.2, R11.1, R13.1, R15.1, R9.1
- net N$5: now also R17.1; no longer U$9.1
- net N$6: now also R18.1; no longer U$10.1
- net N$7: now also R19.1; no longer U$11.1
- net N$8: now also R20.1; no longer U$14.1
- net RUN_BRAKE_1: now also F5.3
- net RUN_BRAKE_2: now also F6.3
- net RUN_BRAKE_3: now also F7.3
- net RUN_BRAKE_4: now also F8.3
- net SPEED_OUT_1: now also SV1.9
- net SPEED_OUT_2: now also SV1.10
- net SPEED_OUT_3: now also SV1.11
- net SPEED_OUT_4: now also SV1.12
- net VRH_1: now also R0.1; no longer U$26.1
Routing:
- net VRH_1: track 123.4 -> 42.6 mm
- net RUN_BRAKE_IN_1: track 0.00 -> 69.0 mm
- net SPEED_1: track 124.0 -> 59.6 mm, vias 0 -> 1
- net RUN_BRAKE_IN_2: track 0.00 -> 61.8 mm, vias 0 -> 1
- net CW_CCW_IN_1: track 31.3 -> 88.9 mm, vias 0 -> 1
- net SPEED_2: track 104.4 -> 48.0 mm, vias 0 -> 1
- net RUN_BRAKE_IN_4: track 0.00 -> 50.7 mm
- net VLM_2: track 120.6 -> 70.5 mm, vias 1 -> 0
- net RUN_BRAKE_IN_3: track 0.00 -> 49.2 mm, vias 0 -> 3
- net VLM_3: track 116.7 -> 77.6 mm, vias 1 -> 0
- net CW_CCW_IN_2: track 41.2 -> 73.4 mm, vias 0 -> 1
- net VLM_1: track 103.2 -> 71.2 mm
- net +5V: track 26.6 -> 5.31 mm
- net SPEED_4: track 60.0 -> 46.4 mm
- net SPEED_3: track 56.5 -> 43.7 mm, vias 2 -> 1
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Other:
- board size 100 x 80 mm -> 100 x 65 mm

Commit message: baitomae
Parts:
- removed CN5: (no value), jst-xa:B14B-XASK-1
- removed SV1: (no value), con-ml:ML26
- added CN6: (no value), jst-xa:B14B-XASK-1
- added R21, R22, R23, R24: (no value), 01_R:1608
- added SV2: (no value), con-ml:ML26
- moved CN1 45.0 mm to (28.0, 55.0)
- moved CN4 45.0 mm to (28.0, 10.0)
- moved F1 45.0 mm to (36.0, 50.0)
- moved F4 45.0 mm to (36.0, 5.00)
- moved F5 45.0 mm to (46.0, 50.0)
- moved F8 45.0 mm to (46.0, 5.00)
- moved LED1 45.0 mm to (7.00, 55.0)
- moved LED4 45.0 mm to (7.00, 10.0)
- moved R1 45.0 mm to (42.0, 47.0)
- moved R10 45.0 mm to (49.0, 54.0)
- moved R15 45.0 mm to (49.0, 5.00)
- moved R16 45.0 mm to (49.0, 9.00)
- moved R2 45.0 mm to (39.0, 50.0)
- moved R7 45.0 mm to (42.0, 2.00)
- moved R8 45.0 mm to (39.0, 5.00)
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Connections:
- new net N$13: LED1.A, R21.1
- new net N$14: LED2.A, R22.1
- new net N$15: LED3.A, R23.1
- new net N$16: LED4.A, R24.1
- net +5V: now also R21.2, R22.2, R23.2, R24.2
- net CW_CCW_IN_1: now also CN6.7, SV2.9; no longer CN5.5, SV1.5
- net CW_CCW_IN_2: now also CN6.8, SV2.10; no longer CN5.6, SV1.6
- net CW_CCW_IN_3: now also CN6.9, SV2.11; no longer CN5.7, SV1.7
- net CW_CCW_IN_4: now also CN6.10, SV2.12; no longer CN5.8, SV1.8
- net GND: now also SV2.1; no longer CN5.13, CN5.14
- net N$5: now also OK1.3, R19.1; no longer OK1.1, R17.1
- net N$6: now also OK1.5; no longer OK1.3
- net N$7: now also OK1.7, R17.1; no longer OK1.5, R19.1
- net N$8: now also OK1.1; no longer OK1.7
- net RUN_BRAKE_IN_1: now also SV2.17; no longer SV1.13
- net RUN_BRAKE_IN_2: now also SV2.18; no longer SV1.14
- net RUN_BRAKE_IN_3: now also SV2.19; no longer SV1.15
- net RUN_BRAKE_IN_4: now also SV2.20; no longer SV1.16
- net SPEED_1: now also OK1.8; no longer OK1.2
- net SPEED_2: now also OK1.6; no longer OK1.4
- net SPEED_3: now also OK1.4; no longer OK1.6
- net SPEED_4: now also OK1.2; no longer OK1.8
- net SPEED_OUT_1: now also CN6.11, OK1.10, SV2.13; no longer CN5.9, OK1.16, SV1.9
- net SPEED_OUT_2: now also CN6.12, OK1.12, SV2.14; no longer CN5.10, OK1.14, SV1.10
- net SPEED_OUT_3: now also CN6.13, OK1.14, SV2.15; no longer CN5.11, OK1.12, SV1.11
- net SPEED_OUT_4: now also CN6.14, OK1.16, SV2.16; no longer CN5.12, OK1.10, SV1.12
- net VLM_1: now also CN6.3, SV2.5; no longer CN5.1, SV1.1
- net VLM_2: now also CN6.4, SV2.6; no longer CN5.2, SV1.2
- net VLM_3: now also CN6.5, SV2.7; no longer CN5.3, SV1.3
- net VLM_4: now also CN6.6, SV2.8; no longer CN5.4, SV1.4
Routing:
- net +5V: track 5.31 -> 140.8 mm, vias 0 -> 2
- net CW_CCW_IN_4: track 65.2 -> 105.0 mm, vias 1 -> 0
- net VLM_4: track 80.3 -> 119.6 mm
- net VRH_1: track 42.6 -> 4.58 mm, vias 1 -> 0
- net CW_CCW_IN_1: track 88.9 -> 53.0 mm
- net RUN_BRAKE_IN_1: track 69.0 -> 50.2 mm
- net RUN_BRAKE_IN_2: track 61.8 -> 46.6 mm, vias 1 -> 2
- net CW_CCW_IN_2: track 73.4 -> 58.5 mm
- net RUN_BRAKE_IN_4: track 50.7 -> 63.9 mm
- net CW_CCW_IN_3: track 59.0 -> 65.5 mm, vias 2 -> 1
- net SPEED_1: track 59.6 -> 54.0 mm
- net N$5: track 2.72 -> 7.70 mm
- net N$15: track 0.00 -> 4.83 mm
- net N$16: track 0.00 -> 4.83 mm
- net N$14: track 0.00 -> 4.83 mm
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- added copper zone on layer 1, net GND

Commit message: kyuukei reset
Connections:
- net +5V: now also CN6.2, SV2.2
Routing:
- net +5V: track 140.8 -> 192.3 mm, vias 2 -> 3
- net SPEED_OUT_1: track 28.1 -> 38.6 mm

Commit message: tetuya
Parts:
- added DRILEGEND: (no value), drilegend:DRILEGEND
Other:
- board text added: "穴図"

Commit message: test2
Parts:
- removed DRILEGEND: (no value), drilegend:DRILEGEND
Connections:
- net +5V: no longer CN6.2, SV2.2
Routing:
- net +5V: track 192.3 -> 140.8 mm, vias 3 -> 2
- net SPEED_OUT_1: track 38.6 -> 28.1 mm
Other:
- board text removed: "穴図"
