File: MyProject/SFT_MoterBridge_1.0v/SFT_MotorBridge.sch (EAGLE design)
At the start: 18 parts

Commit message: 月曜バイト行く前の更新
Parts:
- added SV1: (no value), con-ml:ML26
- added U$10, U$11, U$14, U$26, U$9: (no value), 01_R:RESISTOR__SMD
Connections:
- removed net N$10: CN5.10
- removed net N$11: CN5.11
- removed net N$12: CN5.12
- removed net N$9: CN5.9
- new net +5V: U$10.P$2, U$11.P$2, U$14.P$2, U$26.P$2, U$9.P$2
- new net N$5: OK1A.A, U$9.P$1
- new net N$6: OK1B.A, U$10.P$1
- new net N$7: OK1C.A, U$11.P$1
- new net N$8: OK1D.A, U$14.P$1
- new net SPEED_OUT_1: CN5.9, OK1A.COL
- new net SPEED_OUT_2: CN5.10, OK1B.COL
- new net SPEED_OUT_3: CN5.11, OK1C.COL
- new net SPEED_OUT_4: CN5.12, OK1D.COL
- net CW_CCW_IN_1: now also SV1.5
- net CW_CCW_IN_2: now also SV1.6
- net CW_CCW_IN_3: now also SV1.7
- net CW_CCW_IN_4: now also SV1.8
- net GND: now also OK1A.EMIT, OK1B.EMIT, OK1C.EMIT, OK1D.EMIT
- net SPEED_1: now also OK1A.C
- net SPEED_2: now also OK1B.C
- net SPEED_3: now also OK1C.C
- net SPEED_4: now also OK1D.C
- net VLM_1: now also SV1.1
- net VLM_2: now also SV1.2
- net VLM_3: now also SV1.3
- net VLM_4: now also SV1.4
- net VRH_1: now also U$26.P$1

Commit message: 月曜バイト終了
Parts:
- added F5, F6, F7, F8: CHIP_FET, 06_FET:CHIP_FET
- added LED1, LED2, LED3, LED4: (no value), led:LED5MM
- added R10, R11, R12, R13, R14, R15, R16, R9: (no value), 01_R:RESISTOR__SMD
- renumbered U$10 to R18, U$11 to R19, U$14 to R20, U$26 to R0, U$9 to R17
Connections:
- new net N$10: F6.G, R11.P$2, R12.P$1
- new net N$11: F7.G, R13.P$2, R14.P$1
- new net N$12: F8.G, R15.P$2, R16.P$1
- new net N$9: F5.G, R10.P$1, R9.P$2
- new net RUN_BRAKE_IN_1: R10.P$2, SV1.13
- new net RUN_BRAKE_IN_2: R12.P$2, SV1.14
- new net RUN_BRAKE_IN_3: R14.P$2, SV1.15
- new net RUN_BRAKE_IN_4: R16.P$2, SV1.16
- net ALARM_1: now also LED1.C
- net ALARM_2: now also LED2.C
- net ALARM_3: now also LED3.C
- net ALARM_4: now also LED4.C
- net GND: now also F5.S, F6.S, F7.S, F8.S, R11.P$1, R13.P$1, R15.P$1, R9.P$1
- net RUN_BRAKE_1: now also F5.D
- net RUN_BRAKE_2: now also F6.D
- net RUN_BRAKE_3: now also F7.D
- net RUN_BRAKE_4: now also F8.D
- net SPEED_OUT_1: now also SV1.9
- net SPEED_OUT_2: now also SV1.10
- net SPEED_OUT_3: now also SV1.11
- net SPEED_OUT_4: now also SV1.12

Commit message: baitomae
Parts:
- removed CN5: (no value), jst-xa:B14B-XASK-1
- removed SV1: (no value), con-ml:ML26
- added CN6: (no value), jst-xa:B14B-XASK-1
- added R21, R22, R23, R24: (no value), 01_R:RESISTOR__SMD
- added SV2: (no value), con-ml:ML26
Connections:
- new net N$13: LED1.A, R21.P$1
- new net N$14: LED2.A, R22.P$1
- new net N$15: LED3.A, R23.P$1
- new net N$16: LED4.A, R24.P$1
- net +5V: now also R21.P$2, R22.P$2, R23.P$2, R24.P$2
- net CW_CCW_IN_1: now also CN6.7, SV2.9; no longer CN5.5, SV1.5
- net CW_CCW_IN_2: now also CN6.8, SV2.10; no longer CN5.6, SV1.6
- net CW_CCW_IN_3: now also CN6.9, SV2.11; no longer CN5.7, SV1.7
- net CW_CCW_IN_4: now also CN6.10, SV2.12; no longer CN5.8, SV1.8
- net GND: now also SV2.1; no longer CN5.13, CN5.14
- net N$5: now also OK1B.A, R19.P$1; no longer OK1A.A, R17.P$1
- net N$6: now also OK1C.A; no longer OK1B.A
- net N$7: now also OK1D.A, R17.P$1; no longer OK1C.A, R19.P$1
- net N$8: now also OK1A.A; no longer OK1D.A
- net RUN_BRAKE_IN_1: now also SV2.17; no longer SV1.13
- net RUN_BRAKE_IN_2: now also SV2.18; no longer SV1.14
- net RUN_BRAKE_IN_3: now also SV2.19; no longer SV1.15
- net RUN_BRAKE_IN_4: now also SV2.20; no longer SV1.16
- net SPEED_1: now also OK1D.C; no longer OK1A.C
- net SPEED_2: now also OK1C.C; no longer OK1B.C
- net SPEED_3: now also OK1B.C; no longer OK1C.C
- net SPEED_4: now also OK1A.C; no longer OK1D.C
- net SPEED_OUT_1: now also CN6.11, OK1D.COL, SV2.13; no longer CN5.9, OK1A.COL, SV1.9
- net SPEED_OUT_2: now also CN6.12, OK1C.COL, SV2.14; no longer CN5.10, OK1B.COL, SV1.10
- net SPEED_OUT_3: now also CN6.13, OK1B.COL, SV2.15; no longer CN5.11, OK1C.COL, SV1.11
- net SPEED_OUT_4: now also CN6.14, OK1A.COL, SV2.16; no longer CN5.12, OK1D.COL, SV1.12
- net VLM_1: now also CN6.3, SV2.5; no longer CN5.1, SV1.1
- net VLM_2: now also CN6.4, SV2.6; no longer CN5.2, SV1.2
- net VLM_3: now also CN6.5, SV2.7; no longer CN5.3, SV1.3
- net VLM_4: now also CN6.6, SV2.8; no longer CN5.4, SV1.4
Other:
- moved on the sheet: OK1A, OK1B, OK1C, OK1D

Commit message: kyuukei reset
Connections:
- net +5V: now also CN6.2, SV2.2
Changed lines of the file:
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@@
 <part name="R23" library="01_R" deviceset="RESISTOR__SMD" device=""/>
 <part name="R24" library="01_R" deviceset="RESISTOR__SMD" device=""/>
+<part name="U$26" library="09_OTHER" deviceset="+5V" device=""/>
+<part name="U$35" library="09_OTHER" deviceset="+5V" device=""/>
 </parts>
 <sheets>
@@
 <instance part="R23" gate="G$1" x="63.5" y="10.16" rot="R90"/>
 <instance part="R24" gate="G$1" x="91.44" y="10.16" rot="R90"/>
+<instance part="U$26" gate="G$1" x="154.94" y="12.7"/>
+<instance part="U$35" gate="G$1" x="198.12" y="10.16"/>
 </instances>
 <busses>
@@
 <pinref part="R24" gate="G$1" pin="P$2"/>
 </segment>
-</net>
+<segment>
+<pinref part="CN6" gate="G$1" pin="2"/>
+<pinref part="U$26" gate="G$1" pin="+5V"/>
+</segment>
+<segment>
+<pinref part="SV2" gate="1" pin="2"/>
+<pinref part="U$35" gate="G$1" pin="+5V"/>
+</segment>
+</net>

Commit message: test2
Connections:
- net +5V: no longer CN6.2, SV2.2
Changed lines of the file:
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@@
 <part name="R23" library="01_R" deviceset="RESISTOR__SMD" device=""/>
 <part name="R24" library="01_R" deviceset="RESISTOR__SMD" device=""/>
-<part name="U$26" library="09_OTHER" deviceset="+5V" device=""/>
-<part name="U$35" library="09_OTHER" deviceset="+5V" device=""/>
 </parts>
 <sheets>
@@
 <instance part="R23" gate="G$1" x="63.5" y="10.16" rot="R90"/>
 <instance part="R24" gate="G$1" x="91.44" y="10.16" rot="R90"/>
-<instance part="U$26" gate="G$1" x="154.94" y="12.7"/>
-<instance part="U$35" gate="G$1" x="198.12" y="10.16"/>
 </instances>
 <busses>
@@
 <pinref part="R24" gate="G$1" pin="P$2"/>
 </segment>
-<segment>
-<pinref part="CN6" gate="G$1" pin="2"/>
-<pinref part="U$26" gate="G$1" pin="+5V"/>
-</segment>
-<segment>
-<pinref part="SV2" gate="1" pin="2"/>
-<pinref part="U$35" gate="G$1" pin="+5V"/>
-</segment>
-</net>
+</net>
