File: MyProject/arduino_Pearlite1.0v/Arduino_Micro_Rev03j.brd (EAGLE design)
At the start: 47.8 x 58.3 mm, 46 parts, among them CON1 B3B-ZR, CON2 B3B-ZR, CON3 B3B-ZR, J3 USB-MICRO!!!, J4 3x2M, J5 HEAD17-NOSS, J6 HEAD17-NOSS-1, T1 FDN340P/PMV48XP, T2 PMV48XP, U1 ATMEGA32U4-XUMU, U4 LP2985-33DBVR, Y3 16MHz KX-7

Commit message: syukujitu syuuryou
Parts:
- removed CON1, CON2, CON3: B3B-ZR, jst:B3B-ZR
- removed J3: USB-MICRO!!!, SmartPrj:CON2_USB_MICRO_B_AT
- removed J5: HEAD17-NOSS, SmartPrj:HEAD17-NOSS
- removed J6: HEAD17-NOSS-1, SmartPrj:HEAD17-NOSS-1
- removed RESET: TS42, SmartPrj:TS42
- removed RP3: 22R, resistor-dil:CAY16
- removed U$37: FIDUCIALMOUNT, SmartPrj:FIDUCIA-MOUNT
- removed U$53: FIDUCIAL1X2, SparkFun:FIDUCIAL-1X2
- added A0, A1, A2, A3, A4, A5, CN3, CN4, CN5, CN6: (no value), jst-pa:B3B-PH-K-S
- added CN1, CN7: (no value), jst-pa:B2B-PH-K-S
- added I2C, UART: (no value), jst-pa:B4B-PH-K-S
- added U$33, U$8: (no value), 01_R:1608
- added U$34: MICRO-USB-SHIELD-ZX62R-B-5P, con-hirose1:ZX62R-B-5P
- added U$6: SKRPACE010, 09_1_switch:SKRP
- added U$7: X22, 09_2_CRYSTAL:SMD_X22
- C4: value 1uF -> (none); device SmartPrj:C0402 -> 02_C:1608
- R2: value 10K -> (none); device SmartPrj:R0402 -> 01_R:1608
- moved R2 18.3 mm to (19.0, 8.00), flipped to the top, turned to 0 degrees
- moved D2 13.9 mm to (34.1, 35.8), flipped to the top
- moved ON 12.1 mm to (13.1, 8.42), flipped to the top
- moved J4 3.61 mm to (30.4, 44.1)
- moved C4 2.16 mm to (26.0, 1.50), turned to 180 degrees
- moved R5 2.06 mm to (24.4, 6.32)
- moved U1 1.18 mm to (25.0, 22.0)
- moved C12 0.21 mm to (21.8, 29.6), turned to 270 degrees
Connections:
- removed net 5-GND: RESET.5
- net +5V: now also A0.2, A1.2, A2.2, A3.2, A4.2, A5.2, CN3.2, CN4.2, CN5.2, CN6.2, CN7.2, I2C.2, UART.2; no longer J6.6
- net 3V3: now also C4.P$1; no longer C4.1, J6.16
- net A0: now also A0.3; no longer J6.14
- net A1: now also A1.3; no longer J6.13
- net A2: now also A2.3; no longer J6.12
- net A3: now also A3.3; no longer J6.11
- net A4: now also A4.3; no longer J6.10
- net A5: now also A5.3; no longer J6.9
- net AREF: no longer J6.15
- net D+: now also U$33.1, U$34.3; no longer J3.P3, RP3.8
- net D-: now also U$34.2, U$8.1; no longer J3.P2, RP3.7
- net D0/RX: now also UART.4; no longer J5.4
- net D1/TX: now also UART.3; no longer J5.3
- net D2/SDA: now also I2C.3; no longer J5.7
- net D3/SCL: now also I2C.4; no longer J5.8
- net D4*: now also CN3.3; no longer J5.9
- net D5*: no longer J5.10
- net D6*: now also CN4.3; no longer J5.11
- net D7: no longer J5.12
- net GND: now also A0.1, A1.1, A2.1, A3.1, A4.1, A5.1, C4.P$2, CN3.1, CN4.1, CN5.1, CN6.1, CN7.1, I2C.1, U$34.5, U$34.M1, U$34.M2, U$34.M3, U$34.M4, U$6.3, U$6.4, UART.1; no longer C4.2, J3.P5, J3.S1, J3.S2, J3.S3, J3.S4, J3.S5, J3.S6, J5.6, J6.4, RESET.3, RESET.4, RP3.3, RP3.4, RP3.5, RP3.6
- net IO10*: now also CN6.3; no longer J5.15
- net IO11*: no longer J5.16
- net IO12*: no longer J5.17
- net IO13*: no longer J6.17
- net IO8: no longer J5.13
- net IO9*: now also CN5.3; no longer J5.14
- net MISO: no longer J6.2
- net MOSI: no longer J5.1
- net RD+: now also U$33.2; no longer RP3.1
- net RD-: now also U$8.2; no longer RP3.2
- net RESET: now also U$6.1, U$6.2; no longer J5.5, J6.5, RESET.2
- net RXLED/SS: no longer J5.2
- net SCK: no longer J6.1
- net VIN: no longer J6.3
- net VUSBD: now also U$34.1; no longer J3.P1
Routing:
- net D4*: track 0.00 -> 39.7 mm
- net D1/TX: track 0.00 -> 39.4 mm, vias 0 -> 1
- net D2/SDA: track 0.00 -> 34.2 mm
- net D3/SCL: track 0.00 -> 33.8 mm
- net A5: track 0.00 -> 33.5 mm
- net D6*: track 0.00 -> 32.7 mm
- net IO9*: track 0.00 -> 26.3 mm
- net A0: track 0.00 -> 22.7 mm, vias 0 -> 1
- net IO10*: track 0.00 -> 20.3 mm
- net A1: track 0.00 -> 17.8 mm, vias 0 -> 1
- net A2: track 0.00 -> 13.9 mm
- net +5V: track 0.00 -> 9.49 mm
- net XTAL1: track 0.00 -> 8.46 mm
- net XTAL2: track 0.00 -> 5.18 mm
- net 3V3: track 0.00 -> 4.28 mm
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- added copper zone on layer 1, net +5V
Other:
- board size 47.8 x 58.3 mm -> 50 x 60 mm
- board text removed: "#"
- board text removed: "1"
- board text removed: "2012f"
- board text removed: "3V3"
- board text removed: "A0"
- board text removed: "A1"
- board text removed: "A2"
- board text removed: "A3"
- board text removed: "A4"
- board text removed: "A5"
- board text removed: "Arduino"
- board text removed: "D10"
- board text removed: "D11"
- board text removed: "D12"
- board text removed: "D13"
- board text removed: "D2"
- board text removed: "D3"
- board text removed: "D4"
- board text removed: "D5"
- board text removed: "D6"
- board text removed: "D7"
- board text removed: "D8"
- board text removed: "D9"
- board text removed: "MICRO"
- board text removed: "MISO"
- board text removed: "MOSI"
- board text removed: "NC"
- board text removed: "REF"
- board text removed: "RST"
- board text removed: "RX1"
- board text removed: "SCK"
- board text removed: "SS"
- board text removed: "TM"
- board text removed: "TX1"
- board text removed: "VIN"
- board text removed: "arduino.cc"

Commit message: tetuya
Parts:
- removed Y3: 16MHz KX-7, SmartPrj:CRYSTAL-3.2-2.5
Connections:
- net GND: now also U$7.2, U$7.4; no longer Y3.2, Y3.4
- net XTAL1: now also U$7.1; no longer Y3.3
- net XTAL2: now also U$7.3; no longer Y3.1
Routing:
- net XTAL2: track 5.18 -> 3.95 mm
Changed lines of the file:
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@@
 <attribute name="VALUE" x="21.731" y="6.858" size="1.016" layer="28" rot="MR270"/>
-</element>
-<element name="Y3" library="SmartPrj" package="CRYSTAL-3.2-2.5" value="16MHz KX-7" x="19.318" y="29.845" smashed="yes" rot="R90">
-<attribute name="NAME" x="19.75" y="29.211" size="0.8128" layer="49" ratio="12" rot="R90"/>
-<attribute name="VALUE" x="21.568" y="28.245" size="1.27" layer="27" rot="R90"/>
 </element>
 <element name="U1" library="SmartPrj" package="QFN44ML7X7" value="ATMEGA32U4-XUMU" x="25" y="22" smashed="yes" rot="R225">
@@
 <signal name="XTAL2">
 <contactref element="C12" pad="2"/>
-<contactref element="Y3" pad="1"/>
 <contactref element="U1" pad="16"/>
 <wire x1="23.037778125" y1="24.669325" x2="20.243" y2="27.464103125" width="0.25" layer="1"/>
-<wire x1="20.243" y1="27.464103125" x2="20.243" y2="28.695" width="0.25" layer="1"/>
-<wire x1="20.243" y1="28.695" x2="21.782" y2="29.1595" width="0" layer="19" extent="1-1"/>
+<contactref element="U$7" pad="3"/>
+<wire x1="20.243" y1="27.464103125" x2="21.782" y2="29.1595" width="0" layer="19" extent="1-1"/>
+<wire x1="0.4" y1="-3.3" x2="23.037778125" y2="24.669325" width="0" layer="19" extent="1-1"/>
 </signal>
 <signal name="XTAL1">
 <contactref element="C13" pad="2"/>
-<contactref element="Y3" pad="3"/>
 <contactref element="U1" pad="17"/>
 <wire x1="22.684225" y1="24.315771875" x2="19.3" y2="27.699996875" width="0.25" layer="1"/>
 <wire x1="19.3" y1="27.699996875" x2="19.3" y2="29.9" width="0.25" layer="1"/>
 <wire x1="19.3" y1="29.9" x2="18.393" y2="30.807" width="0.25" layer="1"/>
-<wire x1="18.393" y1="30.807" x2="18.393" y2="30.995" width="0.25" layer="1"/>
-<wire x1="18.393" y1="30.995" x2="18.1115" y2="32.385" width="0" layer="19" extent="1-1"/>
+<contactref element="U$7" pad="1"/>
+<wire x1="18.393" y1="30.807" x2="18.1115" y2="32.385" width="0" layer="19" extent="1-1"/>
+<wire x1="-1.4" y1="-4.7" x2="22.684225" y2="24.315771875" width="0" layer="19" extent="1-1"/>
 </signal>
 <signal name="N$7">
@@
 <contactref element="ON" pad="C"/>
 <contactref element="C14" pad="-"/>
-<contactref element="Y3" pad="2"/>
 <contactref element="U1" pad="15"/>
 <contactref element="U1" pad="EXP"/>
@@
 <contactref element="U1" pad="43"/>
 <contactref element="C3" pad="-"/>
-<contactref element="Y3" pad="4"/>
 <contactref element="C1" pad="2"/>
 <contactref element="R9" pad="1"/>
@@
 <wire x1="23.7" y1="4.375" x2="23.7" y2="5.3" width="0.3" layer="1"/>
 <wire x1="23.7" y1="5.3" x2="23" y2="6" width="0.3" layer="1"/>
-<wire x1="27.1285" y1="30.226" x2="28.0175" y2="28.448" width="0" layer="19" extent="1-1"/>
-<wire x1="19.0005" y1="32.385" x2="18.522" y2="33.655" width="0" layer="19" extent="1-1"/>
+<contactref element="U$7" pad="4"/>
+<contactref element="U$7" pad="2"/>
+<wire x1="44" y1="42" x2="44" y2="52" width="0" layer="19" extent="1-1"/>
+<wire x1="44" y1="32" x2="44" y2="42" width="0" layer="19" extent="1-1"/>
+<wire x1="44" y1="22" x2="44" y2="32" width="0" layer="19" extent="1-1"/>
+<wire x1="44" y1="12" x2="44" y2="22" width="0" layer="19" extent="1-1"/>
+<wire x1="31" y1="54" x2="44" y2="52" width="0" layer="19" extent="1-1"/>
+<wire x1="29.176" y1="46.6405" x2="31" y2="54" width="0" layer="19" extent="1-1"/>
+<wire x1="22.075" y1="45.575" x2="29.176" y2="46.6405" width="0" layer="19" extent="1-1"/>
+<wire x1="22.075" y1="40.425" x2="22.075" y2="45.575" width="0" layer="19" extent="1-1"/>
+<wire x1="24.779" y1="40.1955" x2="22.075" y2="40.425" width="0" layer="19" extent="1-16"/>
+<wire x1="25.3505" y1="38.9382" x2="24.779" y2="40.1955" width="0" layer="19" extent="16-16"/>
+<wire x1="25.3505" y1="37.846" x2="25.3505" y2="38.9382" width="0" layer="19" extent="16-16"/>
+<wire x1="27.573" y1="34.901" x2="25.3505" y2="37.846" width="0" layer="19" extent="1-16"/>
+<wire x1="27.1285" y1="30.226" x2="27.573" y2="34.901" width="0" layer="19" extent="1-1"/>
+<wire x1="28.0175" y1="28.448" x2="27.1285" y2="30.226" width="0" layer="19" extent="1-1"/>
+<wire x1="25.795" y1="26.3525" x2="28.0175" y2="28.448" width="0" layer="19" extent="1-16"/>
+<wire x1="23.89" y1="26.3525" x2="25.795" y2="26.3525" width="0" layer="19" extent="16-16"/>
+<wire x1="23.39133125" y1="25.02288125" x2="23.89" y2="26.3525" width="0" layer="19" extent="1-16"/>
+<wire x1="27.669325" y1="23.96221875" x2="25.795" y2="26.3525" width="0" layer="19" extent="1-16"/>
+<wire x1="27.63969375" y1="21.910690625" x2="27.669325" y2="23.96221875" width="0" layer="19" extent="1-16"/>
 <wire x1="28.7299875" y1="21.0984375" x2="27.63969375" y2="21.910690625" width="0" layer="19" extent="1-16"/>
-<wire x1="23.39133125" y1="25.02288125" x2="23.89" y2="26.3525" width="0" layer="19" extent="1-16"/>
-<wire x1="27.669325" y1="23.96221875" x2="27.63969375" y2="21.910690625" width="0" layer="19" extent="1-16"/>
-<wire x1="27.5095" y1="13.97" x2="24.94" y2="13.97" width="0" layer="19" extent="1-1"/>
 <wire x1="25" y1="22" x2="27.63969375" y2="21.910690625" width="0" layer="19" extent="1-16"/>
-<wire x1="18.393" y1="28.695" x2="20.243" y2="30.995" width="0" layer="19" extent="1-1"/>
 <wire x1="25.901559375" y1="18.270009375" x2="25" y2="22" width="0" layer="19" extent="1-1"/>
 <wire x1="20.91645625" y1="21.451990625" x2="25" y2="22" width="0" layer="19" extent="1-1"/>
+<wire x1="21.782" y1="30.0485" x2="23.89" y2="26.3525" width="0" layer="19" extent="1-16"/>
+<wire x1="19.0005" y1="32.385" x2="21.782" y2="30.0485" width="0" layer="19" extent="1-1"/>
+<wire x1="18.522" y1="33.655" x2="19.0005" y2="32.385" width="0" layer="19" extent="1-1"/>
+<wire x1="18.522" y1="35.56" x2="18.522" y2="33.655" width="0" layer="19" extent="1-1"/>
+<wire x1="24.94" y1="13.97" x2="25.901559375" y2="18.270009375" width="0" layer="19" extent="1-1"/>
+<wire x1="27.5095" y1="13.97" x2="24.94" y2="13.97" width="0" layer="19" extent="1-1"/>
+<wire x1="29.224" y1="8.8265" x2="27.5095" y2="13.97" width="0" layer="19" extent="1-16"/>
+<wire x1="28.208" y1="5.999" x2="29.224" y2="8.8265" width="0" layer="19" extent="16-16"/>
+<wire x1="28.1" y1="3.85" x2="28.208" y2="5.999" width="0" layer="19" extent="1-16"/>
+<wire x1="26.033" y1="6.223" x2="28.208" y2="5.999" width="0" layer="19" extent="16-16"/>
+<wire x1="26.033" y1="7.874" x2="26.033" y2="6.223" width="0" layer="19" extent="16-16"/>
+<wire x1="29.1" y1="1.55" x2="28.1" y2="3.85" width="0" layer="19" extent="1-1"/>
+<wire x1="26.7" y1="1.5" x2="29.1" y2="1.55" width="0" layer="19" extent="1-16"/>
+<wire x1="23.7" y1="5.3" x2="26.033" y2="6.223" width="0" layer="19" extent="1-16"/>
+<wire x1="21.9" y1="3.85" x2="23.7" y2="4.375" width="0" layer="19" extent="1-1"/>
+<wire x1="20.9" y1="1.55" x2="21.9" y2="3.85" width="0" layer="19" extent="1-1"/>
+<wire x1="19.191" y1="3.453" x2="20.9" y2="1.55" width="0" layer="19" extent="1-16"/>
+<wire x1="15" y1="4" x2="19.191" y2="3.453" width="0" layer="19" extent="16-16"/>
+<wire x1="14.16" y1="8.421" x2="15" y2="4" width="0" layer="19" extent="1-1"/>
+<wire x1="18.3" y1="8" x2="14.16" y2="8.421" width="0" layer="19" extent="1-1"/>
+<wire x1="24" y1="57" x2="31" y2="54" width="0" layer="19" extent="1-1"/>
+<wire x1="6" y1="8" x2="14.16" y2="8.421" width="0" layer="19" extent="1-1"/>
+<wire x1="6" y1="18" x2="6" y2="8" width="0" layer="19" extent="1-1"/>
+<wire x1="6" y1="28" x2="6" y2="18" width="0" layer="19" extent="1-1"/>
+<wire x1="6" y1="38" x2="6" y2="28" width="0" layer="19" extent="1-1"/>
+<wire x1="6" y1="48" x2="6" y2="38" width="0" layer="19" extent="1-1"/>
+<wire x1="13" y1="54" x2="6" y2="48" width="0" layer="19" extent="1-1"/>
+<wire x1="-1.4" y1="-3.3" x2="6" y2="8" width="0" layer="19" extent="1-1"/>
+<wire x1="0.4" y1="-4.7" x2="-1.4" y2="-3.3" width="0" layer="19" extent="1-1"/>
 </signal>
 <signal name="D-">

Commit message: test2
Parts:
- removed C4: (no value), 02_C:1608
- removed U$33, U$8: (no value), 01_R:1608
- removed U$6: SKRPACE010, 09_1_switch:SKRP
- removed U$7: X22, 09_2_CRYSTAL:SMD_X22
- removed U4: LP2985-33DBVR, SmartPrj:SOT23-DBV
- added RP3_1, RP3_2: (no value), 01_R:1608
- added SW: SKRPACE010, 09_1_switch:SKRP
- added X1: X22, 09_2_CRYSTAL:SMD_X22
- C1, C10, C11, C2, C6, C9: value 100n -> (none); device SmartPrj:C0402 -> 02_C:1608
- C12, C13: value 22pF -> (none); device SmartPrj:C0402 -> 02_C:1608
- C14, C3: value 22u -> (none); device rcl:SMC_B -> 02_C:3216
- C5, C7: value 1uF -> (none); device SmartPrj:C0402 -> 02_C:1608
- R1, R4, R9: value 10K -> (none); device SmartPrj:R0402 -> 01_R:1608
- R5, R6, R7, R8: value 1K -> (none); device SmartPrj:R0402 -> 01_R:1608
- moved C2 114.9 mm to (0.70, -71.7), flipped to the top, turned to 0 degrees
- moved C1 106.9 mm to (0.70, -66.1), flipped to the top
- moved C9 105.1 mm to (0.70, -75.3), flipped to the top, turned to 0 degrees
- moved R9 102.9 mm to (1.30, -61.0), flipped to the top, turned to 0 degrees
- moved C5 90.0 mm to (0.70, -57.4)
- moved C7 84.8 mm to (0.70, -50.2), turned to 0 degrees
- moved R1 83.5 mm to (1.30, -45.1), turned to 0 degrees
- moved C11 69.3 mm to (0.70, -41.5), flipped to the top, turned to 0 degrees
- moved C6 69.2 mm to (0.70, -53.8), flipped to the top, turned to 0 degrees
- moved C10 68.7 mm to (0.70, -37.9), flipped to the top, turned to 0 degrees
- moved R8 44.1 mm to (1.30, -25.6)
- moved J4 35.5 mm to (17.4, 11.1)
- moved R2 19.9 mm to (38.0, 14.0), turned to 270 degrees
- moved T1 18.2 mm to (25.4, 48.5)
- moved R5 16.9 mm to (7.60, 4.40)
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- renumbered U$34 to USB
Connections:
- removed net 3V3: C4.P$1, U4.5
- net +5V: now also C10.P$1, C11.P$1, C2.P$1, C3.P$1, R1.2, R5.2; no longer C10.1, C11.1, C2.1, C3.+, R1.1, R5.1, U4.1, U4.3
- net +VIN: now also C1.P$1; no longer C1.1
- net AREF: now also C6.P$1; no longer C6.1
- net AVCC: now also C7.P$1; no longer C7.1
- net D+: now also RP3_2.1; no longer U$33.1
- net D-: now also RP3_1.1; no longer U$8.1
- net GND: now also C1.P$2, C10.P$2, C11.P$2, C12.P$1, C13.P$1, C14.P$2, C2.P$2, C3.P$2, C5.P$2, C6.P$2, C7.P$2, C9.P$2, R4.1, SW.3, SW.4, X1.2, X1.4; no longer C1.2, C10.2, C11.2, C12.1, C13.1, C14.-, C2.2, C3.-, C4.P$2, C5.2, C6.2, C7.2, C9.2, R4.2, U$6.3, U$6.4, U$7.2, U$7.4, U4.2
- net HWB: now also R4.2; no longer R4.1
- net IO13*: now also R8.2; no longer R8.1
- net N$2: now also R7.1; no longer R7.2
- net N$3: now also R5.1; no longer R5.2
- net N$4: now also R6.1; no longer R6.2
- net N$7: now also R8.1; no longer R8.2
- net RD+: now also RP3_2.2; no longer U$33.2
- net RD-: now also RP3_1.2; no longer U$8.2
- net RESET: now also R1.1, SW.1, SW.2; no longer R1.2, U$6.1, U$6.2
- net RXLED/SS: now also R7.2; no longer R7.1
- net TXLED: now also R6.2; no longer R6.1
- net UCAP: now also C5.P$1; no longer C5.1
- net VUSB: now also C9.P$1; no longer C9.1
- net VUSBD: now also C14.P$1; no longer C14.+
- net XTAL1: now also C13.P$2, X1.3; no longer C13.2, U$7.1
- net XTAL2: now also C12.P$2, X1.1; no longer C12.2, U$7.3
Routing:
- net D1/TX: track 39.4 -> 0.00 mm, vias 1 -> 0
- net D2/SDA: track 34.2 -> 0.00 mm
- net D3/SCL: track 33.8 -> 0.00 mm
- net A0: track 22.7 -> 0.00 mm, vias 1 -> 0
- net D-: track 0.00 -> 19.5 mm, vias 0 -> 1
- net A1: track 17.8 -> 0.00 mm, vias 1 -> 0
- net D+: track 0.00 -> 14.5 mm, vias 0 -> 1
- net A2: track 13.9 -> 0.00 mm
- net +5V: track 9.49 -> 0.00 mm
- net XTAL1: track 8.27 -> 0.00 mm
- net VUSBD: track 0.00 -> 7.58 mm
- net D6*: track 32.7 -> 25.4 mm, vias 0 -> 1
- net RD-: track 0.00 -> 6.55 mm
- net IO9*: track 26.3 -> 20.8 mm, vias 0 -> 1
- net RD+: track 0.00 -> 5.10 mm
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
Commit message: baito owatta
Parts:
- moved C2 110.8 mm to (13.7, 38.3)
- moved C1 109.8 mm to (13.7, 42.9)
- moved C9 96.7 mm to (40.0, 13.0), turned to 90 degrees
- moved C6 93.6 mm to (33.0, 34.0), flipped to the bottom, turned to 180 degrees
- moved C7 88.0 mm to (37.0, 30.0), turned to 90 degrees
- moved C5 87.8 mm to (31.0, 25.0), flipped to the bottom, turned to 270 degrees
- moved R1 87.7 mm to (37.0, 35.0), turned to 90 degrees
- moved R8 69.1 mm to (23.0, 40.0), flipped to the bottom, turned to 270 degrees
- moved R9 68.6 mm to (20.0, 5.00), flipped to the bottom
- moved C11 53.0 mm to (11.0, 10.5)
- moved T2 49.8 mm to (19.0, 2.00)
- moved T1 46.6 mm to (22.0, 2.00), turned to 270 degrees
- moved C10 46.1 mm to (11.0, 7.00)
- moved L 22.9 mm to (25.0, 36.9), turned to 0 degrees
- moved C13 17.3 mm to (18.0, 20.5), turned to 0 degrees
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Routing:
- net D4*: track 35.8 -> 0.00 mm
- net A5: track 33.9 -> 0.00 mm, vias 1 -> 0
- net D6*: track 25.4 -> 0.00 mm, vias 1 -> 0
- net MISO: track 0.00 -> 24.5 mm
- net SCK: track 0.00 -> 22.2 mm
- net MOSI: track 0.00 -> 22.1 mm, vias 0 -> 1
- net IO10*: track 21.2 -> 0.00 mm, vias 1 -> 0
- net IO9*: track 20.8 -> 0.00 mm, vias 1 -> 0
- net RXLED/SS: track 0.00 -> 20.7 mm, vias 0 -> 1
- net RESET: track 0.00 -> 17.1 mm
- net XTAL1: track 0.00 -> 11.7 mm
- net D+: track 14.5 -> 24.6 mm
- net D-: track 19.5 -> 28.6 mm
- net XTAL2: track 0.00 -> 7.95 mm
- net VUSBD: track 7.58 -> 0.00 mm
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
Commit message: toukyougo
Parts:
- removed SW: SKRPACE010, 09_1_switch:SKRP
- added I2C1: (no value), jst-pa:B4B-PH-K-S
- added RESET: SKRPACE010, 09_1_switch:SKRP
- moved C1 42.3 mm to (18.7, 0.90)
- moved C10 41.0 mm to (41.0, 35.0), turned to 90 degrees
- moved C11 36.5 mm to (38.0, 35.0), turned to 90 degrees
- moved C3 27.3 mm to (14.0, 8.00), flipped to the bottom, turned to 180 degrees
- moved C13 18.1 mm to (13.5, 38.0), turned to 90 degrees
- moved X1 14.6 mm to (16.5, 38.0), turned to 0 degrees
- moved TX 14.4 mm to (12.0, 25.0), turned to 180 degrees
- moved RX 13.9 mm to (15.0, 25.0), turned to 180 degrees
- moved C12 12.6 mm to (16.5, 35.5), turned to 180 degrees
- moved R6 8.94 mm to (12.0, 29.0), turned to 90 degrees
- moved L 8.60 mm to (30.0, 43.9)
- moved C2 8.38 mm to (6.00, 35.0)
- moved R7 8.06 mm to (15.0, 29.0), turned to 90 degrees
- moved C14 8.02 mm to (27.0, 13.5), turned to 90 degrees
- moved C9 5.66 mm to (36.0, 17.0), flipped to the bottom
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Connections:
- net +5V: now also I2C1.2
- net D2/SDA: now also I2C1.3
- net D3/SCL: now also I2C1.4
- net GND: now also I2C1.1, RESET.3, RESET.4; no longer SW.3, SW.4
- net RESET: now also RESET.1, RESET.2; no longer SW.1, SW.2
Routing:
- net +5V: track 0.00 -> 44.2 mm, vias 0 -> 4
- net VUSB: track 0.00 -> 39.3 mm, vias 0 -> 1
- net D-: track 28.6 -> 0.00 mm, vias 1 -> 0
- net D0/RX: track 0.00 -> 27.3 mm
- net D1/TX: track 0.00 -> 24.9 mm, vias 0 -> 1
- net D+: track 24.6 -> 0.00 mm, vias 1 -> 0
- net TXLED: track 0.00 -> 23.4 mm, vias 0 -> 1
- net D2/SDA: track 0.00 -> 21.6 mm, vias 0 -> 1
- net D3/SCL: track 0.00 -> 21.0 mm
- net VUSBD: track 0.00 -> 13.0 mm
- net RXLED/SS: track 20.7 -> 13.1 mm
- net UCAP: track 5.51 -> 0.00 mm
- net GND: track 3.48 -> 0.00 mm
- net RESET: track 17.1 -> 19.7 mm, vias 0 -> 1
- net MISO: track 24.5 -> 26.8 mm
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