File: MyProject/ArduinoMicroShild1.0v/ArduinoMicroShield1.0v.brd (EAGLE design)
At the start: 40 x 65 mm, 30 parts

Commit message: sinnya
Parts:
- added DRILEGEND: (no value), drilegend:DRILEGEND
- moved C2 2.69 mm to (15.0, 8.50), turned to 90 degrees
- turned C1 to 0 degrees
- flipped CN2 to the top
Routing:
- net VIN: track 18.3 -> 14.2 mm
- net +5V: track 16.3 -> 18.0 mm
Other:
- board text added: "ASTAR MINI"
- board text added: "Arduino"
- board text added: "D11"
- board text added: "D12/A11"
- board text added: "D5"
- board text added: "D7"
- board text added: "VIN"
- board text added: "穴図"
