File: MyProject/VideoSelector_2.0v/videoselector_2.0v.brd (EAGLE design)
At the start: 30 x 40 mm, 51 parts, among them CN1 06-JST-B6B-XH-A, CN2 PIN_HEADER_6, IC1 DSPIC33FJ32MC304-PT, IC2 TAR5SB

Commit message: saisin
Parts:
- moved C10 3.00 mm to (20.5, 23.0)
- moved C8 3.00 mm to (20.5, 17.0)
- moved C9 3.00 mm to (20.5, 20.0)
- moved R1 1.46 mm to (18.8, 16.5), turned to 270 degrees
- moved R3 1.06 mm to (18.8, 20.2), turned to 270 degrees
- moved R5 0.79 mm to (18.8, 24.0), turned to 270 degrees
Routing:
- net GND: track 25.2 -> 28.3 mm
- net N$13: track 19.1 -> 21.0 mm
- net N$7: track 26.7 -> 25.6 mm
Other:
- board text added: "+5V"
- board text added: "A"
- board text added: "B"
- board text added: "C"
- board text added: "GND"
