File: MyProject/SK_1.0v/SK_1.0v.brd (EAGLE design)
At the start: 50 x 50 mm, 33 parts, among them CN2 B2B-ZR, CN3 PIN_HEADER_32, CN4 MICRO-USB-SHIELD-ZX62R-B-5P, IC2 MCP73831, IC3 LM2735

Commit message: baito mae hatu
Parts:
- removed CN3: PIN_HEADER_32, 08_CONECTOR:PIN_HEADER_3*2
- removed U$2: CSM-7X-DU, 09_2_CRYSTAL:CSM-7X-DU
- removed U$43, U$44: (no value), 02_C:1608
- added C10, C11, C12, C13: (no value), 02_C:1608
- added IC1: ATMEGA32U4-AU, mega32U4:TQFP44
- added R13, R14: (no value), 01_R:1608
- added U$46: FA-238, 09_2_CRYSTAL:FA-238
- U$3: value ATMEGA32U4-AU -> ICSP; device mega32U4:TQFP44 -> 08_CONECTOR:ICSP
- moved IC3 38.0 mm to (9.00, 36.0), turned to 270 degrees
- moved D1 36.7 mm to (18.5, 45.5)
- moved R8 31.0 mm to (42.0, 14.0), flipped to the bottom, turned to 90 degrees
- moved C1 30.5 mm to (6.50, 33.0), turned to 180 degrees
- moved R1 29.7 mm to (8.50, 25.5), flipped to the bottom, turned to 180 degrees
- moved R10 27.5 mm to (25.5, 35.0)
- moved NCH3 24.6 mm to (37.1, 10.7), turned to 270 degrees
- moved R7 24.6 mm to (40.0, 35.5), turned to 180 degrees
- moved R2 24.5 mm to (12.5, 35.0)
- moved R11 24.3 mm to (28.5, 35.0)
- moved R9 21.5 mm to (39.5, 12.0)
- moved PCH1 19.7 mm to (30.5, 11.5)
- moved R6 18.4 mm to (40.0, 40.0)
- moved NCH1 17.4 mm to (27.2, 39.0)
- moved PCH3 16.1 mm to (37.0, 15.0), turned to 90 degrees
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Connections:
- removed net N$10: R10.2, R11.1
- removed net N$7: NCH1.1
- new net ADC0: IC1.36, R10.2, R11.1
- new net D10: IC1.30, NCH3.3, R9.1
- new net D11: IC1.12, NCH1.1
- new net D13: IC1.32, NCH2.1
- new net MISO: IC1.11, U$3.1
- new net MOSI: IC1.10, U$3.4
- new net N$14: IC1.4, R14.1
- new net N$15: IC1.29
- new net N$16: IC1.28
- new net N$17: IC1.31
- new net N$18: C12.P$2, IC1.6
- new net N$8: IC1.3, R13.1
- new net RESET: IC1.13, U$3.5
- new net SCLK: IC1.9, U$3.3
- net +5V: now also IC1.14, IC1.2, IC1.24, IC1.34, IC1.44; no longer U$3.14, U$3.24, U$3.34, U$3.42, U$3.44
- net +USB5V: now also IC1.7
- net D+: now also R14.2; no longer U$3.4
- net D-: now also R13.2; no longer U$3.3
- net GND: now also C10.P$1, C11.P$1, C12.P$1, C13.P$2, IC1.15, IC1.23, IC1.35, IC1.43, IC1.5, U$3.6, U$46.2, U$46.4; no longer U$3.15, U$3.23, U$3.35, U$3.43, U$43.P$1, U$44.P$1
- net N$11: now also C10.P$2, IC1.17, U$46.1; no longer U$2.2, U$3.17, U$43.P$2
- net N$13: now also C11.P$2, IC1.16, U$46.3; no longer U$2.1, U$3.16, U$44.P$2
- net N$9: now also C13.P$1, IC1.42; no longer NCH3.3, R9.1
Routing:
- net +5V: track 0.00 -> 84.6 mm, vias 0 -> 1
- net +USB5V: track 0.00 -> 46.2 mm, vias 0 -> 3
- net +3.7V: track 0.00 -> 45.1 mm, vias 0 -> 3
- net V2: track 0.00 -> 40.9 mm
- net D11: track 0.00 -> 26.9 mm, vias 0 -> 1
- net D10: track 0.00 -> 25.9 mm, vias 0 -> 1
- net N$14: track 0.00 -> 25.6 mm, vias 0 -> 2
- net N$8: track 0.00 -> 25.4 mm, vias 0 -> 2
- net N$1: track 0.00 -> 15.8 mm
- net N$4: track 0.00 -> 15.7 mm
- net RESET: track 0.00 -> 14.6 mm, vias 0 -> 1
- net SWSIG: track 0.00 -> 11.6 mm
- net N$18: track 0.00 -> 9.48 mm
- net MOSI: track 0.00 -> 8.42 mm
- net N$13: track 0.00 -> 7.74 mm
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- added copper zone on layer 1, net GND
- removed copper zone on layer 1, net N$8

Commit message: hisashiburi
Parts:
- removed CN2: B2B-ZR, jst:B2B-ZR
- removed PCH3: CHIP_FET_P, 06_FET:SOT23
- removed R4, R6, R7: (no value), 01_R:1608
- added C5: 22uF, 02_C:1608
- added C6: 1nF, 02_C:1608
- added C7, C8: 4.7uF, 02_C:1608
- added CN3: (no value), jst-ph:B3B-PH-K-S
- added CN5: (no value), jst-ph:B2B-PH-K-S
- added D2: SOD-123, 15_DIODE:SOD_123
- added R15: 100K, 01_R:1608
- added R16: 30K, 01_R:1608
- added U$31: CSM-7X-DU, 09_2_CRYSTAL:CSM-7X-DU
- added U$37: NEO5MM, 10_LED:NEO5MM
- C1: value (none) -> 22uF
- L1: value D63 -> 22uH
- R1: value (none) -> 2K
- R2: value (none) -> 100K
- R8, R9: value (none) -> 10K
- U$46: value FA-238 -> NEO5MM; device 09_2_CRYSTAL:FA-238 -> 10_LED:NEO5MM
- moved U$46 45.2 mm to (65.0, 35.0), turned to 0 degrees
- moved NCH3 42.3 mm to (32.1, 52.7)
- moved IC3 41.8 mm to (50.0, 28.0), flipped to the bottom
- moved R8 39.4 mm to (36.5, 53.0)
- moved C1 36.8 mm to (43.0, 28.0), flipped to the bottom, turned to 270 degrees
- moved R2 34.2 mm to (46.0, 28.0), flipped to the bottom, turned to 90 degrees
- moved L1 34.2 mm to (49.5, 27.0)
- moved D1 33.2 mm to (49.5, 33.5), turned to 90 degrees
- moved CN4 25.1 mm to (41.0, 14.0)
- moved R9 24.5 mm to (44.5, 36.0), turned to 270 degrees
- moved R13 22.2 mm to (37.5, 25.5), flipped to the bottom
- moved R14 21.4 mm to (34.5, 25.5), flipped to the bottom
- moved NCH1 19.4 mm to (46.5, 36.5)
- moved R10 19.1 mm to (38.5, 49.0), turned to 180 degrees
- moved NCH2 17.8 mm to (46.8, 41.2)
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Connections:
- net N$15 renamed D9
- net N$16 renamed D8
- removed net N$17: IC1.31
- removed net N$5: NCH3.1, PCH3.3, R8.2
- new net A1: IC1.37
- new net A2: IC1.38
- new net A3: CN3.3, IC1.39
- new net A4: IC1.40
- new net A5: IC1.41
- new net D0: IC1.20
- new net D1: IC1.21
- new net D12: IC1.26
- new net D2: IC1.19
- new net D3: IC1.18
- new net D4: IC1.25
- new net D5: IC1.31, NCH1.1
- new net D6: IC1.27
- new net D7: IC1.1
- new net FB: C6.P$2, IC3.3, R15.2, R16.1
- new net HWB: IC1.33
- new net RXLED: IC1.8
- new net STAT: IC2.1
- new net TXLED: IC1.22
- net +3.7V: now also C7.P$1, NCH3.1, R8.2; no longer PCH3.2, R7.2
- net +5V: now also C5.P$1, C6.P$1, CN3.1, CN5.1, D2.C, IC1.7, R16.2; no longer CN2.1
- net +USB5V: now also C8.P$1, D2.A; no longer IC1.7
- net D11: no longer NCH1.1
- net GND: now also C5.P$2, C7.P$2, C8.P$2, CN3.2, CN4.M1, CN4.M2, CN4.M3, CN4.M4, R15.1; no longer R4.1, R6.1, U$46.2, U$46.4
- net N$1: now also CN5.2; no longer CN2.2
- net N$11: now also U$31.2; no longer U$46.1
- net N$13: now also U$31.1; no longer U$46.3
- net N$6: no longer R4.2
- net SWSIG: no longer PCH3.1, R6.2, R7.1
Routing:
- net +3.7V: track 45.1 -> 106.4 mm, vias 3 -> 5
- net V2: track 40.9 -> 70.5 mm, vias 0 -> 1
- net +5V: track 84.6 -> 111.9 mm
- net D11: track 26.9 -> 0.00 mm, vias 1 -> 0
- net +USB5V: track 46.2 -> 30.5 mm, vias 3 -> 1
- net A3: track 0.00 -> 14.0 mm
- net D5: track 0.00 -> 11.4 mm, vias 0 -> 1
- net N$4: track 15.7 -> 5.91 mm, vias 0 -> 1
- net N$14: track 25.6 -> 15.9 mm, vias 2 -> 1
- net FB: track 0.00 -> 8.49 mm
- net GND: track 1.81 -> 10.1 mm, vias 0 -> 1
- net N$5: track 7.22 -> 0.00 mm
- net N$8: track 25.4 -> 19.2 mm, vias 2 -> 1
- net N$11: track 6.30 -> 12.3 mm
- net D+: track 5.13 -> 11.0 mm, vias 0 -> 1
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- added copper zone on layer 1, net N$5
Other:
- board size 50 x 50 mm -> 65.5 x 53 mm
