File: MyProject/SK_test/SK_1.0v.brd (EAGLE design)
At the start: 50 x 50 mm, 28 parts, among them CN2 B2B-ZR, CN4 MICRO-USB-SHIELD-ZX62R-B-5P, IC1 ATMEGA32U4-AU, IC2 MCP73831, IC3 LM2735

Commit message: hisashiburi
Changed lines of the file:
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@@
 <?xml version="1.0" encoding="utf-8"?>
 <!DOCTYPE eagle SYSTEM "eagle.dtd">
-<eagle version="7.3.0">
+<eagle version="7.5.0">
 <drawing>
 <settings>
@@
 <wire x1="48" y1="25.75" x2="48" y2="28.3" width="0.4064" layer="16"/>
 <wire x1="48" y1="28.3" x2="46" y2="30.3" width="0.4064" layer="16"/>
-<via x="43" y="23" extent="1-16" drill="0.6" shape="square"/>
+<via x="43" y="23" extent="1-16" drill="0.5" shape="square"/>
 <wire x1="43" y1="23" x2="45.75" y2="25.75" width="0.4064" layer="16"/>
 <wire x1="45.75" y1="25.75" x2="48" y2="25.75" width="0.4064" layer="16"/>
@@
 <wire x1="6.2" y1="29.95" x2="6.2" y2="30.7" width="0.4" layer="16"/>
 <wire x1="6.2" y1="30.7" x2="7" y2="31.5" width="0.4" layer="16"/>
-<via x="7" y="31.5" extent="1-16" drill="0.6" shape="square"/>
+<via x="7" y="31.5" extent="1-16" drill="0.5" shape="square"/>
 <wire x1="7" y1="31.5" x2="7" y2="32.8" width="0.4" layer="1"/>
 <wire x1="7" y1="32.8" x2="7.2" y2="33" width="0.4" layer="1"/>
 <wire x1="17.5" y1="36.15" x2="17.5" y2="35.5" width="0.4" layer="1"/>
 <wire x1="17.5" y1="35.5" x2="19" y2="34" width="0.4" layer="1"/>
-<via x="19" y="34" extent="1-16" drill="0.6" shape="square"/>
+<via x="19" y="34" extent="1-16" drill="0.5" shape="square"/>
 <wire x1="19" y1="34" x2="31.5" y2="34" width="0.4" layer="16"/>
-<via x="31.5" y="34" extent="1-16" drill="0.6" shape="square"/>
+<via x="31.5" y="34" extent="1-16" drill="0.5" shape="square"/>
 <wire x1="31.5" y1="34" x2="30.2" y2="34" width="0.4" layer="1"/>
 <wire x1="30.2" y1="34" x2="29.2" y2="35" width="0.4" layer="1"/>
@@
 <wire x1="19.3" y1="6.875" x2="19.3" y2="7.8" width="0.4" layer="1"/>
 <wire x1="19.3" y1="7.8" x2="20" y2="8.5" width="0.4" layer="1"/>
-<via x="20" y="8.5" extent="1-16" drill="0.6" shape="square"/>
+<via x="20" y="8.5" extent="1-16" drill="0.5" shape="square"/>
 <wire x1="20" y1="8.5" x2="10.5" y2="8.5" width="0.4" layer="16"/>
 <wire x1="10.5" y1="8.5" x2="8.5" y2="10.5" width="0.4" layer="16"/>
-<via x="8.5" y="10.5" extent="1-16" drill="0.6" shape="square"/>
+<via x="8.5" y="10.5" extent="1-16" drill="0.5" shape="square"/>
 <wire x1="8.5" y1="10.5" x2="8.5" y2="25.5" width="0.4" layer="1"/>
 <wire x1="8.5" y1="25.5" x2="10.5" y2="27.5" width="0.4" layer="1"/>
@@
 <wire x1="8.8" y1="29.95" x2="9.55" y2="29.95" width="0.4" layer="16"/>
 <wire x1="9.55" y1="29.95" x2="10.5" y2="30" width="0.4" layer="16"/>
-<via x="10.5" y="30" extent="1-16" drill="0.6" shape="square"/>
+<via x="10.5" y="30" extent="1-16" drill="0.5" shape="square"/>
 <wire x1="10.5" y1="30" x2="10.5" y2="27.5" width="0.4" layer="1"/>
 </signal>
@@
 <wire x1="30.5" y1="16" x2="28.5" y2="18" width="0.4064" layer="16"/>
 <wire x1="28.5" y1="18" x2="28.5" y2="25.5" width="0.4064" layer="16"/>
-<via x="28.5" y="25.5" extent="1-16" drill="0.6" shape="square"/>
+<via x="28.5" y="25.5" extent="1-16" drill="0.5" shape="square"/>
 <wire x1="28.5" y1="25.5" x2="29.6" y2="26.6" width="0.4064" layer="1"/>
 <wire x1="29.6" y1="26.6" x2="30.8" y2="26.6" width="0.4064" layer="1"/>
@@
 <contactref element="R13" pad="1"/>
 <wire x1="19.5" y1="13.2" x2="19.5" y2="14.5" width="0.4064" layer="1"/>
-<via x="19.5" y="14.5" extent="1-16" drill="0.6" shape="square"/>
+<via x="19.5" y="14.5" extent="1-16" drill="0.5" shape="square"/>
 <wire x1="19.5" y1="14.5" x2="19.5" y2="28.5" width="0.4064" layer="16"/>
 <wire x1="19.5" y1="28.5" x2="16.5" y2="31.5" width="0.4064" layer="16"/>
-<via x="16.5" y="31.5" extent="1-16" drill="0.6" shape="square"/>
+<via x="16.5" y="31.5" extent="1-16" drill="0.5" shape="square"/>
 <wire x1="16.5" y1="31.5" x2="16.5" y2="29" width="0.4064" layer="1"/>
 <wire x1="16.5" y1="29" x2="18.1" y2="27.4" width="0.4064" layer="1"/>
@@
 <contactref element="R14" pad="1"/>
 <wire x1="17.5" y1="13.2" x2="17.5" y2="14.5" width="0.4064" layer="1"/>
-<via x="17.5" y="14.5" extent="1-16" drill="0.6" shape="square"/>
+<via x="17.5" y="14.5" extent="1-16" drill="0.5" shape="square"/>
 <wire x1="17.5" y1="14.5" x2="17.5" y2="27" width="0.4064" layer="16"/>
-<via x="15" y="30" extent="1-16" drill="0.6" shape="square"/>
+<via x="15" y="30" extent="1-16" drill="0.5" shape="square"/>
 <wire x1="19.2" y1="26.6" x2="17.9" y2="26.6" width="0.4064" layer="1"/>
 <wire x1="17.9" y1="26.6" x2="15" y2="29.5" width="0.4064" layer="1"/>
@@
 <wire x1="21.8" y1="17.8" x2="21.5" y2="17.5" width="0.4064" layer="1"/>
 <wire x1="21.5" y1="17.5" x2="16" y2="17.5" width="0.4064" layer="1"/>
-<via x="16" y="17.5" extent="1-16" drill="0.6" shape="square"/>
+<via x="16" y="17.5" extent="1-16" drill="0.5" shape="square"/>
 <wire x1="16" y1="17.5" x2="16" y2="22.31" width="0.4064" layer="16"/>
 <wire x1="16" y1="22.31" x2="14.27" y2="24.04" width="0.4064" layer="16"/>
@@
 <wire x1="30.8" y1="22.6" x2="32.1" y2="22.6" width="0.4064" layer="1"/>
 <wire x1="32.1" y1="22.6" x2="32.5" y2="23" width="0.4064" layer="1"/>
-<via x="32.5" y="23" extent="1-16" drill="0.6" shape="square"/>
+<via x="32.5" y="23" extent="1-16" drill="0.5" shape="square"/>
 <wire x1="32.5" y1="23" x2="32.5" y2="30.5" width="0.4064" layer="16"/>
 <wire x1="32.5" y1="30.5" x2="30" y2="33" width="0.4064" layer="16"/>
